File: pcb/linecard/phy0_mdi.kicad_sch (KiCad schematic)
At the start: 99 parts, among them J2 LPJG47036AWNL, J5 LPJG47036AWNL, U10 VSC8512, U11 ESD224DQAR, U12 ESD224DQAR, U13 ESD224DQAR, U14 ESD224DQAR, U15 ESD224DQAR, U16 ESD224DQAR, U17 ESD224DQAR, U18 ESD224DQAR, U19 ESD224DQAR, U20 ESD224DQAR, U21 ESD224DQAR, U22 ESD224DQAR, U23 ESD224DQAR, U24 ESD224DQAR, U25 ESD224DQAR, U26 ESD224DQAR, U27 ESD224DQAR, U28 ESD224DQAR, U29 ESD224DQAR, U30 ESD224DQAR, U31 ESD224DQAR, U32 ESD224DQAR, U33 ESD224DQAR, U34 ESD224DQAR

Commit message: Finished initial schematic of line card
Parts:
- C193, C194, C195, C196, C197, C198, C199, C200, C201, C202, C203, C204, C205, C206, C207, C208, C209, C210, C211, C212, C213, C214, C215, C216, C217, C218, C219, C220, C221, C222, C223, C224, C225, C226, C227, C228, C229, C230, C231, C232, C233, C234, C235, C236, C237, C238, C239, C240: value C -> 0.1 uF; footprint (none) -> azonenberg_pcb:EIA_0402_CAP_NOSILK
- R31, R32, R33, R34, R35, R36, R37, R38, R39, R40, R41, R42, R43, R44, R45, R46, R47, R48, R49, R50, R51, R52, R53, R54: value R -> 470
- U10: footprint (none) -> azonenberg_pcb:BGA_676_27x27_FULLARRAY_1MM_FFG676
Other:
- note removed: "TODO: port number indexes on 8-11"

Commit message: Finished initial schematic review
Parts:
- J2, J5: footprint (none) -> azonenberg_pcb:CONN_LINKPP_LPJG47036AWNL
- U11, U12, U13, U14, U15, U16, U17, U18, U19, U20, U21, U22, U23, U24, U25, U26, U27, U28, U29, U30, U31, U32, U33, U34: footprint (none) -> azonenberg_pcb:DFN_10_0.5MM_2.5x1MM_TI_DQA
Connections:
- net CHGND: now also J2.SHLD, J2.SHLD, J2.SHLD, J2.SHLD, J2.SHLD, J2.SHLD, J2.SHLD, J2.SHLD, J5.SHLD; no longer J2.A0 (SHLD), J2.B0 (SHLD), J2.C0 (SHLD), J2.D0 (SHLD), J2.E0 (SHLD), J2.F0 (SHLD), J2.G0 (SHLD), J2.H0 (SHLD), J5.D0 (SHLD)
- net PHY0_D1_P: now also U11.6 (IO4_S); no longer U11.5 (IO4_S)
- net PHY0_D3_P: now also U12.6 (IO4_S); no longer U12.5 (IO4_S)
- net PHY10_D1_P: now also U31.6 (IO4_S); no longer U31.5 (IO4_S)
- net PHY10_D3_P: now also U32.6 (IO4_S); no longer U32.5 (IO4_S)
- net PHY11_D1_P: now also U33.6 (IO4_S); no longer U33.5 (IO4_S)
- net PHY11_D3_P: now also U34.6 (IO4_S); no longer U34.5 (IO4_S)
- net PHY1_D1_P: now also U13.6 (IO4_S); no longer U13.5 (IO4_S)
- net PHY1_D3_P: now also U14.6 (IO4_S); no longer U14.5 (IO4_S)
- net PHY2_D1_P: now also U15.6 (IO4_S); no longer U15.5 (IO4_S)
- net PHY2_D3_P: now also U16.6 (IO4_S); no longer U16.5 (IO4_S)
- net PHY3_D1_P: now also U17.6 (IO4_S); no longer U17.5 (IO4_S)
- net PHY3_D3_P: now also U18.6 (IO4_S); no longer U18.5 (IO4_S)
- net PHY4_D1_P: now also U19.6 (IO4_S); no longer U19.5 (IO4_S)
- net PHY4_D3_P: now also U20.6 (IO4_S); no longer U20.5 (IO4_S)
- net PHY5_D1_P: now also U21.6 (IO4_S); no longer U21.5 (IO4_S)
- net PHY5_D3_P: now also U22.6 (IO4_S); no longer U22.5 (IO4_S)
- net PHY6_D1_P: now also U23.6 (IO4_S); no longer U23.5 (IO4_S)
- net PHY6_D3_P: now also U24.6 (IO4_S); no longer U24.5 (IO4_S)
- net PHY7_D1_P: now also U25.6 (IO4_S); no longer U25.5 (IO4_S)
- net PHY7_D3_P: now also U26.6 (IO4_S); no longer U26.5 (IO4_S)
- net PHY8_D1_P: now also U27.6 (IO4_S); no longer U27.5 (IO4_S)
- net PHY8_D3_P: now also U28.6 (IO4_S); no longer U28.5 (IO4_S)
- net PHY9_D1_P: now also U29.6 (IO4_S); no longer U29.5 (IO4_S)
- net PHY9_D3_P: now also U30.6 (IO4_S); no longer U30.5 (IO4_S)

Commit message: Began layout of first few ports and left VSC8512
Connections:
- net PHY0_D1_N: now also U11.6 (IO4_S); no longer U11.7 (IO3_S)
- net PHY0_D1_P: now also U11.7 (IO3_S); no longer U11.6 (IO4_S)
- net PHY0_D2_N: now also U12.9 (IO2_S); no longer U12.10 (IO1_S)
- net PHY0_D2_P: now also U12.10 (IO1_S); no longer U12.9 (IO2_S)
- net PHY0_M1_N: now also U11.5 (IO4_C); no longer U11.4 (IO3_C)
- net PHY0_M1_P: now also U11.4 (IO3_C); no longer U11.5 (IO4_C)
- net PHY0_M2_N: now also U12.2 (IO2_C); no longer U12.1 (IO1_C)
- net PHY0_M2_P: now also U12.1 (IO1_C); no longer U12.2 (IO2_C)
- net PHY1_D0_N: now also U14.7 (IO3_S); no longer U13.10 (IO1_S)
- net PHY1_D0_P: now also U14.6 (IO4_S); no longer U13.9 (IO2_S)
- net PHY1_D1_N: now also U14.9 (IO2_S); no longer U13.7 (IO3_S)
- net PHY1_D1_P: now also U14.10 (IO1_S); no longer U13.6 (IO4_S)
- net PHY1_D2_N: now also U13.10 (IO1_S); no longer U14.10 (IO1_S)
- net PHY1_D2_P: now also U13.9 (IO2_S); no longer U14.9 (IO2_S)
- net PHY1_D3_N: now also U13.6 (IO4_S); no longer U14.7 (IO3_S)
- net PHY1_D3_P: now also U13.7 (IO3_S); no longer U14.6 (IO4_S)
- net PHY1_M0_N: now also U14.4 (IO3_C); no longer U13.1 (IO1_C)
- net PHY1_M0_P: now also U14.5 (IO4_C); no longer U13.2 (IO2_C)
- net PHY1_M1_N: now also U14.2 (IO2_C); no longer U13.4 (IO3_C)
- net PHY1_M1_P: now also U14.1 (IO1_C); no longer U13.5 (IO4_C)
- net PHY1_M2_N: now also U13.1 (IO1_C); no longer U14.1 (IO1_C)
- net PHY1_M2_P: now also U13.2 (IO2_C); no longer U14.2 (IO2_C)
- net PHY1_M3_N: now also U13.5 (IO4_C); no longer U14.4 (IO3_C)
- net PHY1_M3_P: now also U13.4 (IO3_C); no longer U14.5 (IO4_C)
- net PHY2_D0_N: now also U15.7 (IO3_S); no longer U15.10 (IO1_S)
- net PHY2_D0_P: now also U15.6 (IO4_S); no longer U15.9 (IO2_S)
- net PHY2_D1_N: now also U16.10 (IO1_S); no longer U15.7 (IO3_S)
- net PHY2_D1_P: now also U16.9 (IO2_S); no longer U15.6 (IO4_S)
- net PHY2_D2_N: now also U16.6 (IO4_S); no longer U16.10 (IO1_S)
- net PHY2_D2_P: now also U16.7 (IO3_S); no longer U16.9 (IO2_S)
- net PHY2_D3_N: now also U15.9 (IO2_S); no longer U16.7 (IO3_S)
- net PHY2_D3_P: now also U15.10 (IO1_S); no longer U16.6 (IO4_S)
- net PHY2_M0_N: now also U15.4 (IO3_C); no longer U15.1 (IO1_C)
- net PHY2_M0_P: now also U15.5 (IO4_C); no longer U15.2 (IO2_C)
- net PHY2_M1_N: now also U16.1 (IO1_C); no longer U15.4 (IO3_C)
- net PHY2_M1_P: now also U16.2 (IO2_C); no longer U15.5 (IO4_C)
- net PHY2_M2_N: now also U16.5 (IO4_C); no longer U16.1 (IO1_C)
- net PHY2_M2_P: now also U16.4 (IO3_C); no longer U16.2 (IO2_C)
- net PHY2_M3_N: now also U15.2 (IO2_C); no longer U16.4 (IO3_C)
- net PHY2_M3_P: now also U15.1 (IO1_C); no longer U16.5 (IO4_C)
- net PHY3_D0_N: now also U18.7 (IO3_S); no longer U17.10 (IO1_S)
- net PHY3_D0_P: now also U18.6 (IO4_S); no longer U17.9 (IO2_S)
- net PHY3_D1_N: now also U17.10 (IO1_S); no longer U17.7 (IO3_S)
- net PHY3_D1_P: now also U17.9 (IO2_S); no longer U17.6 (IO4_S)
- net PHY3_D2_N: now also U17.6 (IO4_S); no longer U18.10 (IO1_S)
- net PHY3_D2_P: now also U17.7 (IO3_S); no longer U18.9 (IO2_S)
- net PHY3_D3_N: now also U18.9 (IO2_S); no longer U18.7 (IO3_S)
- net PHY3_D3_P: now also U18.10 (IO1_S); no longer U18.6 (IO4_S)
- net PHY3_M0_N: now also U18.4 (IO3_C); no longer U17.1 (IO1_C)
- net PHY3_M0_P: now also U18.5 (IO4_C); no longer U17.2 (IO2_C)
- net PHY3_M1_N: now also U17.1 (IO1_C); no longer U17.4 (IO3_C)
- net PHY3_M1_P: now also U17.2 (IO2_C); no longer U17.5 (IO4_C)
- net PHY3_M2_N: now also U17.5 (IO4_C); no longer U18.1 (IO1_C)
- net PHY3_M2_P: now also U17.4 (IO3_C); no longer U18.2 (IO2_C)
- net PHY3_M3_N: now also U18.2 (IO2_C); no longer U18.4 (IO3_C)
- net PHY3_M3_P: now also U18.1 (IO1_C); no longer U18.5 (IO4_C)
Changed lines of the file:
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@@
 	)
 	(label "PHY3_D1_N"
-		(at 102.87 195.58 180)
+		(at 102.87 190.5 180)
 		(fields_autoplaced yes)
 		(effects
@@
 	)
 	(label "PHY1_D0_P"
-		(at 102.87 82.55 180)
+		(at 102.87 110.49 180)
 		(fields_autoplaced yes)
 		(effects
@@
 	)
 	(label "PHY1_D1_P"
-		(at 102.87 87.63 180)
+		(at 102.87 102.87 180)
 		(fields_autoplaced yes)
 		(effects
@@
 	)
 	(label "PHY1_M1_N"
-		(at 123.19 85.09 0)
+		(at 123.19 105.41 0)
 		(fields_autoplaced yes)
 		(effects
@@
 	)
 	(label "PHY1_D2_N"
-		(at 102.87 102.87 180)
+		(at 102.87 80.01 180)
 		(fields_autoplaced yes)
 		(effects
@@
 	)
 	(label "PHY2_D1_N"
-		(at 102.87 139.7 180)
+		(at 102.87 157.48 180)
 		(fields_autoplaced yes)
 		(effects
@@
 	)
 	(label "PHY2_M3_P"
-		(at 123.19 165.1 0)
+		(at 123.19 134.62 0)
 		(fields_autoplaced yes)
 		(effects
@@
 	)
 	(label "PHY1_M1_P"
-		(at 123.19 87.63 0)
+		(at 123.19 102.87 0)
 		(fields_autoplaced yes)
 		(effects
@@
 	)
 	(label "PHY1_M3_N"
-		(at 123.19 107.95 0)
+		(at 123.19 87.63 0)
 		(fields_autoplaced yes)
 		(effects
@@
 	)
 	(label "PHY2_M0_N"
-		(at 123.19 134.62 0)
+		(at 123.19 139.7 0)
 		(fields_autoplaced yes)
 		(effects
@@
 	)
 	(label "PHY0_M1_N"
-		(at 123.19 29.21 0)
+		(at 123.19 31.75 0)
 		(fields_autoplaced yes)
 		(effects
@@
 	)
 	(label "PHY3_M1_N"
-		(at 123.19 195.58 0)
+		(at 123.19 190.5 0)
 		(fields_autoplaced yes)
 		(effects
@@
 	)
 	(label "PHY2_M1_P"
-		(at 123.19 142.24 0)
+		(at 123.19 160.02 0)
 		(fields_autoplaced yes)
 		(effects
@@
 	)
 	(label "PHY2_M1_N"
-		(at 123.19 139.7 0)
+		(at 123.19 157.48 0)
 		(fields_autoplaced yes)
 		(effects
@@
 	)
 	(label "PHY3_M0_N"
-		(at 123.19 190.5 0)
+		(at 123.19 218.44 0)
 		(fields_autoplaced yes)
 		(effects
@@
 	)
 	(label "PHY3_D0_P"
-		(at 102.87 193.04 180)
+		(at 102.87 220.98 180)
 		(fields_autoplaced yes)
 		(effects
@@
 	)
 	(label "PHY3_D3_P"
-		(at 102.87 220.98 180)
+		(at 102.87 213.36 180)
 		(fields_autoplaced yes)
 		(effects
@@
 	)
 	(label "PHY2_D1_P"
-		(at 102.87 142.24 180)
+		(at 102.87 160.02 180)
 		(fields_autoplaced yes)
 		(effects
@@
 	)
 	(label "PHY2_M0_P"
-		(at 123.19 137.16 0)
+		(at 123.19 142.24 0)
 		(fields_autoplaced yes)
 		(effects
@@
 	)
 	(label "PHY3_D2_N"
-		(at 102.87 213.36 180)
+		(at 102.87 198.12 180)
 		(fields_autoplaced yes)
 		(effects
@@
 	)
 	(label "PHY2_M2_P"
-		(at 123.19 160.02 0)
+		(at 123.19 162.56 0)
 		(fields_autoplaced yes)
 		(effects
@@
 	)
 	(label "PHY2_D3_P"
-		(at 102.87 165.1 180)
+		(at 102.87 134.62 180)
 		(fields_autoplaced yes)
 		(effects
@@
 	)
 	(label "PHY1_M0_P"
-		(at 123.19 82.55 0)
+		(at 123.19 110.49 0)
 		(fields_autoplaced yes)
 		(effects
@@
 	)
 	(label "PHY3_M1_P"
-		(at 123.19 198.12 0)
+		(at 123.19 193.04 0)
 		(fields_autoplaced yes)
 		(effects
@@
 	)
 	(label "PHY3_M3_N"
-		(at 123.19 218.44 0)
+		(at 123.19 215.9 0)
 		(fields_autoplaced yes)
 		(effects
@@
 	)
 	(label "PHY0_M2_N"
-		(at 123.19 46.99 0)
+		(at 123.19 49.53 0)
 		(fields_autoplaced yes)
 		(effects
@@
 	)
 	(label "PHY2_D0_N"
-		(at 102.87 134.62 180)
+		(at 102.87 139.7 180)
 		(fields_autoplaced yes)
 		(effects
@@
 	)
 	(label "PHY3_M2_P"
-		(at 123.19 215.9 0)
+		(at 123.19 195.58 0)
 		(fields_autoplaced yes)
 		(effects
@@
 	)
 	(label "PHY2_M3_N"
-		(at 123.19 162.56 0)
+		(at 123.19 137.16 0)
 		(fields_autoplaced yes)
 		(effects
@@
 	)
 	(label "PHY1_M2_N"
-		(at 123.19 102.87 0)
+		(at 123.19 80.01 0)
 		(fields_autoplaced yes)
 		(effects
@@
 	)
 	(label "PHY3_D1_P"
-		(at 102.87 198.12 180)
+		(at 102.87 193.04 180)
 		(fields_autoplaced yes)
 		(effects
@@
 	)
 	(label "PHY1_D2_P"
-		(at 102.87 105.41 180)
+		(at 102.87 82.55 180)
 		(fields_autoplaced yes)
 		(effects
@@
 	)
 	(label "PHY2_D2_P"
-		(at 102.87 160.02 180)
+		(at 102.87 162.56 180)
 		(fields_autoplaced yes)
 		(effects
@@
 	)
 	(label "PHY2_D2_N"
-		(at 102.87 157.48 180)
+		(at 102.87 165.1 180)
 		(fields_autoplaced yes)
 		(effects
@@
 	)
 	(label "PHY0_D1_N"
-		(at 102.87 29.21 180)
+		(at 102.87 31.75 180)
 		(fields_autoplaced yes)
 		(effects
@@
 	)
 	(label "PHY1_D3_P"
-		(at 102.87 110.49 180)
+		(at 102.87 85.09 180)
 		(fields_autoplaced yes)
 		(effects
@@
 	)
 	(label "PHY0_D1_P"
-		(at 102.87 31.75 180)
+		(at 102.87 29.21 180)
 		(fields_autoplaced yes)
 		(effects
@@
 	)
 	(label "PHY1_D3_N"
-		(at 102.87 107.95 180)
+		(at 102.87 87.63 180)
 		(fields_autoplaced yes)
 		(effects
@@
 	)
 	(label "PHY2_D3_N"
-		(at 102.87 162.56 180)
+		(at 102.87 137.16 180)
 		(fields_autoplaced yes)
 		(effects
@@
 	)
 	(label "PHY1_M0_N"
-		(at 123.19 80.01 0)
+		(at 123.19 107.95 0)
 		(fields_autoplaced yes)
 		(effects
@@
 	)
 	(label "PHY3_M3_P"
-		(at 123.19 220.98 0)
+		(at 123.19 213.36 0)
 		(fields_autoplaced yes)
 		(effects
@@
 	)
 	(label "PHY1_M3_P"
-		(at 123.19 110.49 0)
+		(at 123.19 85.09 0)
 		(fields_autoplaced yes)
 		(effects
@@
 	)
 	(label "PHY3_M2_N"
-		(at 123.19 213.36 0)
+		(at 123.19 198.12 0)
 		(fields_autoplaced yes)
 		(effects
@@
 	)
 	(label "PHY3_D3_N"
-		(at 102.87 218.44 180)
+		(at 102.87 215.9 180)
 		(fields_autoplaced yes)
 		(effects
@@
 	)
 	(label "PHY1_D0_N"
-		(at 102.87 80.01 180)
+		(at 102.87 107.95 180)
 		(fields_autoplaced yes)
 		(effects
@@
 	)
 	(label "PHY3_D0_N"
-		(at 102.87 190.5 180)
+		(at 102.87 218.44 180)
 		(fields_autoplaced yes)
 		(effects
@@
 	)
 	(label "PHY3_D2_P"
-		(at 102.87 215.9 180)
+		(at 102.87 195.58 180)
 		(fields_autoplaced yes)
 		(effects
@@
 	)
 	(label "PHY1_D1_N"
-		(at 102.87 85.09 180)
+		(at 102.87 105.41 180)
 		(fields_autoplaced yes)
 		(effects
@@
 	)
 	(label "PHY2_D0_P"
-		(at 102.87 137.16 180)
+		(at 102.87 142.24 180)
 		(fields_autoplaced yes)
 		(effects
@@
 	)
 	(label "PHY0_D2_P"
-		(at 102.87 49.53 180)
+		(at 102.87 46.99 180)
 		(fields_autoplaced yes)
 		(effects
@@
 	)
 	(label "PHY0_M2_P"
-		(at 123.19 49.53 0)
+		(at 123.19 46.99 0)
 		(fields_autoplaced yes)
 		(effects
@@
 	)
 	(label "PHY0_D2_N"
-		(at 102.87 46.99 180)
+		(at 102.87 49.53 180)
 		(fields_autoplaced yes)
 		(effects
@@
 	)
 	(label "PHY3_M0_P"
-		(at 123.19 193.04 0)
+		(at 123.19 220.98 0)
 		(fields_autoplaced yes)
 		(effects
@@
 	)
 	(label "PHY0_M1_P"
-		(at 123.19 31.75 0)
+		(at 123.19 29.21 0)
 		(fields_autoplaced yes)
 		(effects
@@
 	)
 	(label "PHY1_M2_P"
-		(at 123.19 105.41 0)
+		(at 123.19 82.55 0)
 		(fields_autoplaced yes)
 		(effects
@@
 	)
 	(label "PHY2_M2_N"
-		(at 123.19 157.48 0)
+		(at 123.19 165.1 0)
 		(fields_autoplaced yes)
 		(effects

Commit message: Update waiting for new part from vendor
Connections:
- net PHY1_D0_N: now also U14.10 (IO1_S); no longer U14.7 (IO3_S)
- net PHY1_D0_P: now also U14.9 (IO2_S); no longer U14.6 (IO4_S)
- net PHY1_D1_N: now also U14.7 (IO3_S); no longer U14.9 (IO2_S)
- net PHY1_D1_P: now also U14.6 (IO4_S); no longer U14.10 (IO1_S)
- net PHY1_D2_N: now also U13.9 (IO2_S); no longer U13.10 (IO1_S)
- net PHY1_D2_P: now also U13.10 (IO1_S); no longer U13.9 (IO2_S)
- net PHY1_D3_N: now also U13.7 (IO3_S); no longer U13.6 (IO4_S)
- net PHY1_D3_P: now also U13.6 (IO4_S); no longer U13.7 (IO3_S)
- net PHY1_M0_N: now also U14.1 (IO1_C); no longer U14.4 (IO3_C)
- net PHY1_M0_P: now also U14.2 (IO2_C); no longer U14.5 (IO4_C)
- net PHY1_M1_N: now also U14.4 (IO3_C); no longer U14.2 (IO2_C)
- net PHY1_M1_P: now also U14.5 (IO4_C); no longer U14.1 (IO1_C)
- net PHY1_M2_N: now also U13.2 (IO2_C); no longer U13.1 (IO1_C)
- net PHY1_M2_P: now also U13.1 (IO1_C); no longer U13.2 (IO2_C)
- net PHY1_M3_N: now also U13.4 (IO3_C); no longer U13.5 (IO4_C)
- net PHY1_M3_P: now also U13.5 (IO4_C); no longer U13.4 (IO3_C)
- net PHY2_D2_N: now also U15.9 (IO2_S); no longer U16.6 (IO4_S)
- net PHY2_D2_P: now also U15.10 (IO1_S); no longer U16.7 (IO3_S)
- net PHY2_D3_N: now also U16.6 (IO4_S); no longer U15.9 (IO2_S)
- net PHY2_D3_P: now also U16.7 (IO3_S); no longer U15.10 (IO1_S)
- net PHY2_M2_N: now also U15.2 (IO2_C); no longer U16.5 (IO4_C)
- net PHY2_M2_P: now also U15.1 (IO1_C); no longer U16.4 (IO3_C)
- net PHY2_M3_N: now also U16.5 (IO4_C); no longer U15.2 (IO2_C)
- net PHY2_M3_P: now also U16.4 (IO3_C); no longer U15.1 (IO1_C)
Changed lines of the file:
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@@
 	)
 	(label "PHY1_D0_P"
-		(at 102.87 110.49 180)
+		(at 102.87 105.41 180)
 		(fields_autoplaced yes)
 		(effects
@@
 	)
 	(label "PHY1_D1_P"
-		(at 102.87 102.87 180)
+		(at 102.87 110.49 180)
 		(fields_autoplaced yes)
 		(effects
@@
 	)
 	(label "PHY1_M1_N"
-		(at 123.19 105.41 0)
+		(at 123.19 107.95 0)
 		(fields_autoplaced yes)
 		(effects
@@
 	)
 	(label "PHY1_D2_N"
-		(at 102.87 80.01 180)
+		(at 102.87 82.55 180)
 		(fields_autoplaced yes)
 		(effects
@@
 	)
 	(label "PHY2_M3_P"
-		(at 123.19 134.62 0)
+		(at 123.19 162.56 0)
 		(fields_autoplaced yes)
 		(effects
@@
 	)
 	(label "PHY1_M1_P"
-		(at 123.19 102.87 0)
+		(at 123.19 110.49 0)
 		(fields_autoplaced yes)
 		(effects
@@
 	)
 	(label "PHY1_M3_N"
-		(at 123.19 87.63 0)
+		(at 123.19 85.09 0)
 		(fields_autoplaced yes)
 		(effects
@@
 	)
 	(label "PHY2_M2_P"
-		(at 123.19 162.56 0)
+		(at 123.19 134.62 0)
 		(fields_autoplaced yes)
 		(effects
@@
 	)
 	(label "PHY2_D3_P"
-		(at 102.87 134.62 180)
+		(at 102.87 162.56 180)
 		(fields_autoplaced yes)
 		(effects
@@
 	)
 	(label "PHY1_M0_P"
-		(at 123.19 110.49 0)
+		(at 123.19 105.41 0)
 		(fields_autoplaced yes)
 		(effects
@@
 	)
 	(label "PHY2_M3_N"
-		(at 123.19 137.16 0)
+		(at 123.19 165.1 0)
 		(fields_autoplaced yes)
 		(effects
@@
 	)
 	(label "PHY1_M2_N"
-		(at 123.19 80.01 0)
+		(at 123.19 82.55 0)
 		(fields_autoplaced yes)
 		(effects
@@
 	)
 	(label "PHY1_D2_P"
-		(at 102.87 82.55 180)
+		(at 102.87 80.01 180)
 		(fields_autoplaced yes)
 		(effects
@@
 	)
 	(label "PHY2_D2_P"
-		(at 102.87 162.56 180)
+		(at 102.87 134.62 180)
 		(fields_autoplaced yes)
 		(effects
@@
 	)
 	(label "PHY2_D2_N"
-		(at 102.87 165.1 180)
+		(at 102.87 137.16 180)
 		(fields_autoplaced yes)
 		(effects
@@
 	)
 	(label "PHY1_D3_P"
-		(at 102.87 85.09 180)
+		(at 102.87 87.63 180)
 		(fields_autoplaced yes)
 		(effects
@@
 	)
 	(label "PHY1_D3_N"
-		(at 102.87 87.63 180)
+		(at 102.87 85.09 180)
 		(fields_autoplaced yes)
 		(effects
@@
 	)
 	(label "PHY2_D3_N"
-		(at 102.87 137.16 180)
+		(at 102.87 165.1 180)
 		(fields_autoplaced yes)
 		(effects
@@
 	)
 	(label "PHY1_M0_N"
-		(at 123.19 107.95 0)
+		(at 123.19 102.87 0)
 		(fields_autoplaced yes)
 		(effects
@@
 	)
 	(label "PHY1_M3_P"
-		(at 123.19 85.09 0)
+		(at 123.19 87.63 0)
 		(fields_autoplaced yes)
 		(effects
@@
 	)
 	(label "PHY1_D0_N"
-		(at 102.87 107.95 180)
+		(at 102.87 102.87 180)
 		(fields_autoplaced yes)
 		(effects
@@
 	)
 	(label "PHY1_D1_N"
-		(at 102.87 105.41 180)
+		(at 102.87 107.95 180)
 		(fields_autoplaced yes)
 		(effects
@@
 	)
 	(label "PHY1_M2_P"
-		(at 123.19 82.55 0)
+		(at 123.19 80.01 0)
 		(fields_autoplaced yes)
 		(effects
@@
 	)
 	(label "PHY2_M2_N"
-		(at 123.19 165.1 0)
+		(at 123.19 137.16 0)
 		(fields_autoplaced yes)
 		(effects
