File: pcb/linecard/phy0_mdi.kicad_sch (KiCad schematic)
At the start: 51 parts, among them J2 LPJT476156AENL, J5 LPJT476156AENL, U10 VSC8512, U11 ESD224DQAR, U12 ESD224DQAR, U13 ESD224DQAR, U14 ESD224DQAR, U15 ESD224DQAR, U16 ESD224DQAR, U17 ESD224DQAR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

Commit message: Added software workaround for line card LED1 errata
Other:
- note added: "ERRATA: LED1 even/odd are swapped"
Changed lines of the file:
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@@
+		)
+	)
+	(text "ERRATA: LED1 even/odd are swapped"
+		(exclude_from_sim no)
+		(at 20.574 242.824 0)
+		(effects
+			(font
+				(size 1.27 1.27)
+			)
+			(justify left)
 		)
 	)
