File: pcb/linecard/phy1.kicad_sch (KiCad schematic)
At the start: 33 parts, among them J11 SMPM, J12 SMPM, J13 XILINX_JTAG, M13 960-27-12-D-AB-0, U35 VSC8512, U61 SIT9121AC-2B2-33E125.000000

Commit message: Finished initial schematic review
Parts:
- added TP24: TESTPOINT, symbol conn:CONN_01X01
- J14: value ~ -> ARF6-08-S-D-A-K-TR; footprint (none) -> azonenberg_pcb:CONN_SAMTEC_ARF6-08-S-D-A-K-TR
- R92: value 10K -> 1K
Connections:
- net GND: now also J14.27 (SHLD)
- net at U35.R2 (MDINT): now also TP24.1 (P1)
- no-connect marks 43 -> 42
Other:
- moved on the sheet: C467, C468, C469, C470, C471, C472, C473, C474, C475, C476, C477, C478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

Commit message: Began layout of first few ports and left VSC8512
Parts:
- TP24: footprint (none) -> azonenberg_pcb:TESTPOINT_SMT_0.5MM
Changed lines of the file:
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@@
 			)
 		)
-		(property "Footprint" ""
+		(property "Footprint" "azonenberg_pcb:TESTPOINT_SMT_0.5MM"
 			(at 67.31 189.23 0)
 			(effects
