File: pcb/linecard/linecard.kicad_sch (KiCad schematic)
At the start: 17 parts, among them M1 LONGTHING, M10 SCREWHOLE, M11 SCREWHOLE, M2 OSHW, M3 WEEE, M4 SCREWHOLE, M5 SCREWHOLE, M6 SCREWHOLE, M7 SCREWHOLE, M8 SCREWHOLE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

Commit message: Updating file: linecard.kicad_pcb with current fully routed design
Parts:
- removed TP21, TP4: GROUNDCLIP, azonenberg_pcb:TESTPOINT_SMT_KEYSTONE_5016, symbol conn:CONN_01X01
Changed lines of the file:
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@@
-	)
-	(junction
-		(at 20.32 265.43)
-		(diameter 0)
-		(color 0 0 0 0)
 	)
 	(junction
@@
 	)
 	(junction
-		(at 20.32 270.51)
-		(diameter 0)
-		(color 0 0 0 0)
-	)
-	(junction
 		(at 48.26 210.82)
 		(diameter 0)
@@
 	(wire
 		(pts
-			(xy 20.32 265.43) (xy 20.32 270.51)
+			(xy 21.59 204.47) (xy 21.59 210.82)
+		)
+		(stroke
+			(width 0)
+			(type default)
+		)
+	)
+	(polyline
+		(pts
+			(xy 12.7 199.39) (xy 74.93 199.39)
 		)
 		(stroke
@@
 	(wire
 		(pts
-			(xy 21.59 204.47) (xy 21.59 210.82)
+			(xy 48.26 210.82) (xy 48.26 217.17)
+		)
+		(stroke
+			(width 0)
+			(type default)
+		)
+	)
+	(wire
+		(pts
+			(xy 48.26 204.47) (xy 48.26 210.82)
 		)
 		(stroke
@@
 	(polyline
 		(pts
-			(xy 12.7 199.39) (xy 74.93 199.39)
+			(xy 74.93 255.27) (xy 74.93 284.48)
+		)
+		(stroke
+			(width 0)
+			(type default)
+		)
+	)
+	(polyline
+		(pts
+			(xy 74.93 229.87) (xy 74.93 199.39)
 		)
 		(stroke
@@
 	(wire
 		(pts
-			(xy 48.26 210.82) (xy 48.26 217.17)
+			(xy 67.31 20.32) (xy 82.55 20.32)
 		)
 		(stroke
@@
 	(wire
 		(pts
-			(xy 48.26 204.47) (xy 48.26 210.82)
+			(xy 48.26 217.17) (xy 48.26 223.52)
+		)
+		(stroke
+			(width 0)
+			(type default)
+		)
+	)
+	(wire
+		(pts
+			(xy 21.59 210.82) (xy 21.59 217.17)
 		)
 		(stroke
@@
 	(polyline
 		(pts
-			(xy 74.93 255.27) (xy 74.93 284.48)
+			(xy 12.7 229.87) (xy 74.93 229.87)
+		)
+		(stroke
+			(width 0)
+			(type default)
+		)
+	)
+	(wire
+		(pts
+			(xy 67.31 27.94) (xy 82.55 27.94)
+		)
+		(stroke
+			(width 0)
+			(type default)
+		)
+	)
+	(wire
+		(pts
+			(xy 20.32 260.35) (xy 20.32 265.43)
 		)
 		(stroke
@@
 	(polyline
 		(pts
-			(xy 74.93 229.87) (xy 74.93 199.39)
+			(xy 12.7 255.27) (xy 74.93 255.27)
 		)
 		(stroke
@@
 	(wire
 		(pts
-			(xy 67.31 20.32) (xy 82.55 20.32)
+			(xy 21.59 217.17) (xy 21.59 223.52)
 		)
 		(stroke
@@
 	(wire
 		(pts
-			(xy 48.26 217.17) (xy 48.26 223.52)
-		)
-		(stroke
-			(width 0)
-			(type default)
-		)
-	)
-	(wire
-		(pts
-			(xy 21.59 210.82) (xy 21.59 217.17)
-		)
-		(stroke
-			(width 0)
-			(type default)
-		)
-	)
-	(polyline
-		(pts
-			(xy 12.7 229.87) (xy 74.93 229.87)
-		)
-		(stroke
-			(width 0)
-			(type default)
-		)
-	)
-	(wire
-		(pts
-			(xy 67.31 27.94) (xy 82.55 27.94)
-		)
-		(stroke
-			(width 0)
-			(type default)
-		)
-	)
-	(wire
-		(pts
-			(xy 20.32 260.35) (xy 20.32 265.43)
-		)
-		(stroke
-			(width 0)
-			(type default)
-		)
-	)
-	(polyline
-		(pts
-			(xy 12.7 255.27) (xy 74.93 255.27)
-		)
-		(stroke
-			(width 0)
-			(type default)
-		)
-	)
-	(wire
-		(pts
-			(xy 21.59 217.17) (xy 21.59 223.52)
-		)
-		(stroke
-			(width 0)
-			(type default)
-		)
-	)
-	(wire
-		(pts
 			(xy 67.31 25.4) (xy 82.55 25.4)
-		)
-		(stroke
-			(width 0)
-			(type default)
-		)
-	)
-	(wire
-		(pts
-			(xy 20.32 270.51) (xy 20.32 275.59)
 		)
 		(stroke
@@
 					(unit 1)
 				)
-			)
-		)
-	)
-	(symbol
-		(lib_id "conn:CONN_01X01")
-		(at 25.4 275.59 0)
-		(unit 1)
-		(exclude_from_sim no)
-		(in_bom yes)
-		(on_board yes)
-		(dnp no)
-		(fields_autoplaced yes)
-		(property "Reference" "TP21"
-			(at 27.305 274.7553 0)
-			(effects
-				(font
-					(size 1.27 1.27)
-				)
-				(justify left)
-			)
-		)
-		(property "Value" "GROUNDCLIP"
-			(at 27.305 277.2922 0)
-			(effects
-				(font
-					(size 1.27 1.27)
-				)
-				(justify left)
-			)
-		)
-		(property "Footprint" "azonenberg_pcb:TESTPOINT_SMT_KEYSTONE_5016"
-			(at 25.4 275.59 0)
-			(effects
-				(font
-					(size 1.27 1.27)
-				)
-				(hide yes)
-			)
-		)
-		(property "Datasheet" ""
-			(at 25.4 275.59 0)
-			(effects
-				(font
-					(size 1.27 1.27)
-				)
-				(hide yes)
-			)
-		)
-		(property "Description" ""
-			(at 25.4 275.59 0)
-			(effects
-				(font
-					(size 1.27 1.27)
-				)
-				(hide yes)
-			)
-		)
-		(pin "1"
-		)
-		(instances
-			(project "linecard"
-				(path "/a55ad1ec-4cad-4d06-8b73-31c98dcc1d79"
-					(reference "TP21")
-					(unit 1)
-				)
-			)
-		)
-	)
-	(symbol
-		(lib_id "conn:CONN_01X01")
-		(at 25.4 270.51 0)
-		(unit 1)
-		(exclude_from_sim no)
-		(in_bom yes)
-		(on_board yes)
-		(dnp no)
-		(fields_autoplaced yes)
-		(property "Reference" "TP4"
-			(at 27.305 269.6753 0)
-			(effects
-				(font
-					(size 1.27 1.27)
-				)
-				(justify left)
-			)
-		)
-		(property "Value" "GROUNDCLIP"
-			(at 27.305 272.2122 0)
-			(effects
-				(font
-					(size 1.27 1.27)
-				)
-				(justify left)
-			)
-		)
-		(property "Footprint" "azonenberg_pcb:TESTPOINT_SMT_KEYSTONE_5016"
-			(at 25.4 270.51 0)
-			(effects
-				(font
-					(size 1.27 1.27)
-				)
-				(hide yes)
-			)
-		)
-		(property "Datasheet" ""
-			(at 25.4 270.51 0)
-			(effects
-				(font
-					(size 1.27 1.27)
-				)
-				(hide yes)
-			)
-		)
-		(property "Description" ""
-			(at 25.4 270.51 0)
-			(effects
-				(font
-					(size 1.27 1.27)
-				)
-				(hide yes)
-			)
-		)
-		(pin "1"
-		)
-		(instances
-			(project "linecard"
-				(path "/a55ad1ec-4cad-4d06-8b73-31c98dcc1d79"
-					(reference "TP4")
-					(unit 1)
-				)
