File: pcb/linecard/phy1_mdi.kicad_sch (KiCad schematic)
At the start: 51 parts, among them J5 LPJT476156AENL, J9 LPJT476156AENL, U35 VSC8512, U36 ESD224DQAR, U37 ESD224DQAR, U38 ESD224DQAR, U39 ESD224DQAR, U40 ESD224DQAR, U41 ESD224DQAR, U42 ESD224DQAR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

Commit message: Added software workaround for line card LED1 errata
Other:
- note added: "ERRATA: LED1 even/odd are swapped"
Changed lines of the file:
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@@
+		)
+	)
+	(text "ERRATA: LED1 even/odd are swapped"
+		(exclude_from_sim no)
+		(at 16.764 240.538 0)
+		(effects
+			(font
+				(size 1.27 1.27)
+			)
+			(justify left)
 		)
 	)
