File: pcb/linecard/psu.kicad_sch (KiCad schematic)
At the start: 103 parts, among them J1 CONN_ATX12V, J3 CORTEX_DEBUG_ETM, J4 0532611071, SW1 SWITCH, SW2 SWITCH, U1 MYMGK00504ERSR, U2 MYMGK00504ERSR, U3 MYMGK00504ERSR, U4 MYMGK00504ERSR, U5 STM32L431-QFN48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

Commit message: Continued tying up loose ends on routing of left side and supervisor
Connections:
- net 1V0_2_EN: now also U5.28 (PB15); no longer U5.11 (PA1)
- net 1V0_2_PGOOD: now also U5.29 (PA8); no longer U5.32 (PA11)
- net 1V0_EN: now also U5.26 (PB13); no longer U5.10 (PA0)
- net 1V0_PGOOD: now also U5.27 (PB14); no longer U5.33 (PA12)
- net 2V5_EN: now also U5.32 (PA11); no longer U5.12 (PA2)
- net 2V5_PGOOD: now also U5.33 (PA12); no longer U5.18 (PB0)
- net 3V3_PGOOD: now also U5.25 (PB12); no longer U5.13 (PA3)
- net INA_ALERT: now also U5.11 (PA1); no longer U5.28 (PB15)
- net PHY0_RST: now also U5.10 (PA0); no longer U5.26 (PB13)
- net PHY1_RST: now also U5.12 (PA2); no longer U5.27 (PB14)
- net SOFT_RST: now also U5.13 (PA3); no longer U5.25 (PB12)
Changed lines of the file:
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@@
 	(title_block
 		(title "LATENTRED Line Card")
-		(date "2024-12-17")
+		(date "2024-12-18")
 		(rev "0.1")
 		(company "Antikernel Labs")
@@
 	)
 	(no_connect
+		(at 251.46 115.57)
+	)
+	(no_connect
 		(at 364.49 87.63)
 	)
@@
 	)
 	(no_connect
-		(at 200.66 135.89)
-	)
-	(no_connect
 		(at 251.46 128.27)
 	)
@@
 	)
 	(label "1V0_2_PGOOD"
-		(at 200.66 143.51 180)
+		(at 200.66 135.89 180)
 		(fields_autoplaced yes)
 		(effects
@@
 	)
 	(label "1V0_EN"
-		(at 200.66 115.57 180)
+		(at 251.46 148.59 180)
 		(fields_autoplaced yes)
 		(effects
@@
 	)
 	(label "1V0_PGOOD"
-		(at 200.66 146.05 180)
+		(at 251.46 151.13 180)
 		(fields_autoplaced yes)
 		(effects
@@
 	)
 	(label "1V0_2_EN"
-		(at 200.66 118.11 180)
+		(at 251.46 153.67 180)
 		(fields_autoplaced yes)
 		(effects
@@
 	)
 	(label "3V3_PGOOD"
-		(at 200.66 123.19 180)
+		(at 251.46 146.05 180)
 		(fields_autoplaced yes)
 		(effects
@@
 	)
 	(label "2V5_PGOOD"
-		(at 251.46 115.57 180)
+		(at 200.66 146.05 180)
 		(fields_autoplaced yes)
 		(effects
@@
 	)
 	(label "INA_ALERT"
-		(at 251.46 153.67 180)
+		(at 200.66 118.11 180)
 		(fields_autoplaced yes)
 		(effects
@@
 	)
 	(label "SOFT_RST"
-		(at 251.46 146.05 180)
+		(at 200.66 123.19 180)
 		(fields_autoplaced yes)
 		(effects
@@
 	)
 	(label "2V5_EN"
-		(at 200.66 120.65 180)
+		(at 200.66 143.51 180)
 		(fields_autoplaced yes)
 		(effects
@@
 	(hierarchical_label "PHY1_RST"
 		(shape output)
-		(at 251.46 151.13 180)
+		(at 200.66 120.65 180)
 		(fields_autoplaced yes)
 		(effects
@@
 	(hierarchical_label "PHY0_RST"
 		(shape output)
-		(at 251.46 148.59 180)
+		(at 200.66 115.57 180)
 		(fields_autoplaced yes)
 		(effects

Commit message: Added planes, more LED signals, etc
Connections:
- net FAULT_LED: now also U5.12 (PA2); no longer U5.45 (PB8)
- net INA_ALERT: now also U5.3 (PC14); no longer U5.11 (PA1)
- net PHY0_PWRDN: now also U5.2 (PC13); no longer U5.5 (PH0)
- net PHY0_RST: now also U5.46 (PB9); no longer U5.10 (PA0)
- net PHY1_PWRDN: now also U5.18 (PB0); no longer U5.6 (PH1)
- net PHY1_RST: now also U5.19 (PB1); no longer U5.12 (PA2)
- net PWRGOOD_LED: now also U5.10 (PA0); no longer U5.46 (PB9)
- net SYSOK_LED: now also U5.11 (PA1); no longer U5.21 (PB10)
- net TEMP_ALERT: now also U5.45 (PB8); no longer U5.19 (PB1)
Changed lines of the file:
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@@
 	)
 	(no_connect
-		(at 364.49 82.55)
+		(at 195.58 170.18)
 	)
 	(no_connect
-		(at 195.58 179.07)
+		(at 195.58 167.64)
 	)
 	(no_connect
-		(at 251.46 115.57)
+		(at 364.49 82.55)
 	)
 	(no_connect
@@
 	)
 	(no_connect
-		(at 195.58 181.61)
-	)
-	(no_connect
 		(at 251.46 128.27)
 	)
@@
 	)
 	(no_connect
+		(at 251.46 140.97)
+	)
+	(no_connect
 		(at 364.49 90.17)
 	)
@@
 	)
 	(label "FAULT_LED"
-		(at 251.46 135.89 180)
+		(at 200.66 120.65 180)
 		(fields_autoplaced yes)
 		(effects
@@
 	)
 	(label "TEMP_ALERT"
-		(at 251.46 118.11 180)
+		(at 251.46 135.89 180)
 		(fields_autoplaced yes)
 		(effects
@@
 	)
 	(label "INA_ALERT"
-		(at 200.66 118.11 180)
+		(at 195.58 181.61 180)
 		(fields_autoplaced yes)
 		(effects
@@
 	)
 	(label "SYSOK_LED"
-		(at 251.46 140.97 180)
+		(at 200.66 118.11 180)
 		(fields_autoplaced yes)
 		(effects
@@
 	)
 	(label "PWRGOOD_LED"
-		(at 251.46 138.43 180)
+		(at 200.66 115.57 180)
 		(fields_autoplaced yes)
 		(effects
@@
 	(hierarchical_label "PHY1_PWRDN"
 		(shape input)
-		(at 195.58 170.18 180)
+		(at 251.46 115.57 180)
 		(fields_autoplaced yes)
 		(effects
@@
 	(hierarchical_label "PHY1_RST"
 		(shape output)
-		(at 200.66 120.65 180)
+		(at 251.46 118.11 180)
 		(fields_autoplaced yes)
 		(effects
@@
 	(hierarchical_label "PHY0_RST"
 		(shape output)
-		(at 200.66 115.57 180)
+		(at 251.46 138.43 180)
 		(fields_autoplaced yes)
 		(effects
@@
 	(hierarchical_label "PHY0_PWRDN"
 		(shape input)
-		(at 195.58 167.64 180)
+		(at 195.58 179.07 180)
 		(fields_autoplaced yes)
 		(effects

Commit message: Continued power routing on right PHY
Connections:
- net SOFT_PWR: now also U5.21 (PB10); no longer U5.22 (PB11)
- net SOFT_RST: now also U5.22 (PB11); no longer U5.13 (PA3)
Changed lines of the file:
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@@
 	)
 	(no_connect
-		(at 251.46 140.97)
+		(at 200.66 123.19)
 	)
 	(no_connect
@@
 	)
 	(label "SOFT_PWR"
-		(at 251.46 143.51 180)
+		(at 251.46 140.97 180)
 		(fields_autoplaced yes)
 		(effects
@@
 	)
 	(label "SOFT_RST"
-		(at 200.66 123.19 180)
+		(at 251.46 143.51 180)
 		(fields_autoplaced yes)
 		(effects

Commit message: More routing cleanup
Connections:
- net TEMP_ALERT: now also U5.41 (PB5); no longer U5.45 (PB8)
Changed lines of the file:
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@@
 	(title_block
 		(title "LATENTRED Line Card")
-		(date "2024-12-19")
+		(date "2024-12-21")
 		(rev "0.1")
 		(company "Antikernel Labs")
@@
 	)
 	(no_connect
-		(at 251.46 128.27)
-	)
-	(no_connect
 		(at 364.49 80.01)
 	)
@@
 	)
 	(no_connect
+		(at 251.46 135.89)
+	)
+	(no_connect
 		(at 364.49 90.17)
 	)
@@
 	)
 	(label "TEMP_ALERT"
-		(at 251.46 135.89 180)
+		(at 251.46 128.27 180)
 		(fields_autoplaced yes)
 		(effects

Commit message: Line card: fixed typo in component value and alternate pinmux mode
Parts:
- C11: value 22 uF 25VC -> 22 uF 25V
Changed lines of the file:
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@@
 	(title_block
 		(title "LATENTRED Line Card")
-		(date "2024-12-21")
-		(rev "0.1")
+		(date "2025-05-20")
+		(rev "0.1b")
 		(company "Antikernel Labs")
 		(comment 1 "Andrew D. Zonenberg")
@@
 			)
 		)
-		(property "Value" "22 uF 25VC"
+		(property "Value" "22 uF 25V"
 			(at 33.401 190.4421 0)
 			(effects
