File: pcb/pdu/pdu.kicad_pcb (KiCad board)
At the start: 4 copper layers, 105 x 47 mm, 46 parts, among them J1 CONN_PCIE_PWR_8PIN, J2 MOLEX_0039291087, J3 MOLEX_0039291048, J4 MOLEX_0039291048, J5 CONN_IBC_MGMT_DEVICE, J6 CONN_IBC_MGMT_HOST, M1 LOGO, M2 LOGO, M3 LOGO, M4 LOGO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

Commit message: Finished PDU design, ready for fab
Parts:
- C3: moved to F.Cu
- moved M2 36.9 mm to (92.0, 69.5)
- moved M3 29.6 mm to (113.0, 69.5)
- moved C12 0.20 mm to (143.6, 69.6)
Routing:
- net /12V0_LC1: track 13.8 -> 15.2 mm
- net /3V3_SB: track 176.2 -> 176.8 mm
- net /I2C_SDA: track 150.9 -> 151.4 mm
Other:
- board text added: "S/N"
