File: pcb/lcbringup/arf6.kicad_sch (KiCad schematic)
At the start: 13 parts, among them J10 SMPM, J11 ARF6-08-S-D-A-K-TR, J12 SMPM, J13 SMPM, J14 SMPM, J15 SMPM, J16 SMPM, J17 SMPM, J18 SMPM, J19 SMPM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

Commit message: Continued lcbringup layout on ARF6 area
Changed lines of the file:
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@@
 	(title_block
 		(title "Andrew D. Zonenberg")
-		(date "2025-01-14")
+		(date "2025-01-19")
 		(rev "0.1")
 		(company "Antikernel Labs")
@@
 	)
 	(label "GND"
-		(at 111.76 26.67 180)
-		(fields_autoplaced yes)
-		(effects
-			(font
-				(size 1.27 1.27)
-			)
-			(justify right bottom)
-		)
-	)
-	(label "GND"
 		(at 60.96 88.9 0)
 		(fields_autoplaced yes)
@@
 		)
 	)
+	(hierarchical_label "GND"
+		(shape input)
+		(at 111.76 26.67 180)
+		(fields_autoplaced yes)
+		(effects
+			(font
+				(size 1.27 1.27)
+			)
+			(justify right)
+		)
+	)
