File: pcb/lcbringup/fpgasupport.kicad_sch (KiCad schematic)
At the start: 42 parts, among them J1 XILINX_JTAG, U1 XC7A35T-2FGG484C

Commit message: Continued lcbringup layout
Parts:
- added C60, C61: 4.7 uF, azonenberg_pcb:EIA_0603_CAP_NOSILK, symbol device:C
- added C62, C63, C67, C92: 0.47 uF, azonenberg_pcb:EIA_0402_CAP_NOSILK, symbol device:C
Connections:
- net 3V3: now also C60.1, C61.1, C62.1, C63.1, C67.1, C92.1
- net GND: now also C60.2, C61.2, C62.2, C63.2, C67.2, C92.2
Other:
- note added: "3V3 VCCO (reduced since we're only using some IO banks)"
- note removed: "3V3 VCCO (reduced since we're only using 1-2 banks of IO)"
- moved on the sheet: C13, C14, C5, C6, C7, C8

Commit message: Conitnued lcbringup layout, power supply is now floorplanned
Parts:
- added C100, C101, C98, C99: 0.47 uF, azonenberg_pcb:EIA_0402_CAP_NOSILK, symbol device:C
- added C96, C97: 4.7 uF, azonenberg_pcb:EIA_0603_CAP_NOSILK, symbol device:C
Connections:
- net 3V3: no longer U1.AA17 (VCCO_13), U1.AB14 (VCCO_13), U1.V16 (VCCO_13), U1.W13 (VCCO_13), U1.Y10 (VCCO_13)
- net GND: now also C100.2, C101.2, C96.2, C97.2, C98.2, C99.2
- new net 2V5: C100.1, C101.1, C96.1, C97.1, C98.1, C99.1, U1.AA17 (VCCO_13), U1.AB14 (VCCO_13), U1.V16 (VCCO_13), U1.W13 (VCCO_13), U1.Y10 (VCCO_13)
Other:
- note added: "2V5 VCCO (reduced since we're only using two pins for slow MDIO)"
- note added: "FIXME FIXME NEED LVCMOS25 FOR MDIO"
- moved on the sheet: C13, C14, C5, C6, C7, C8

Commit message: Finished lcbringup, ready to order
Other:
- note removed: "FIXME FIXME NEED LVCMOS25 FOR MDIO"
Changed lines of the file:
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@@
 	(title_block
 		(title "Andrew D. Zonenberg")
-		(date "2025-01-19")
+		(date "2025-01-20")
 		(rev "0.1")
 		(company "Antikernel Labs")
@@
 		)
 	)
-	(text "FIXME FIXME NEED LVCMOS25 FOR MDIO"
-		(exclude_from_sim no)
-		(at 179.07 193.04 0)
-		(effects
-			(font
-				(size 1.27 1.27)
-			)
-		)
-	)
