File: pcb/lcbringup/mcu.kicad_sch (KiCad schematic)
At the start: 71 parts, among them J4 CORTEX_DEBUG_ETM, J5 CONN_01X03, J6 CONN_01X03, U1 XC7A35T-2FGG484C, U2 STM32H735-UFBGA176-25, U4 ECS-1612MV-250-CN, U6 ECS-1612MV-250-CN, U7 AT24MAC402

Commit message: Continued lcbringup layout
Parts:
- removed C60: 4.7 uF, azonenberg_pcb:EIA_0603_CAP_NOSILK, symbol device:C
- removed C61, C62, C63, C67: 0.47 uF, azonenberg_pcb:EIA_0402_CAP_NOSILK, symbol device:C
- removed D6, D7, D8, D9: GREEN, azonenberg_pcb:EIA_0402_LED, symbol device:LED
- removed J6: CONN_01X03, azonenberg_pcb:CONN_HEADER_2.54MM_1x3, symbol conn:CONN_01X03
- removed R12, R13, R14, R15: 33K, azonenberg_pcb:EIA_0402_RES_NOSILK, symbol device:R
- removed R25: 33, azonenberg_pcb:EIA_0402_RES_NOSILK, symbol device:R
- removed U6: ECS-1612MV-250-CN, azonenberg_pcb:OSCILLATOR_1.6x1.2, symbol osc-azonenberg:OSC
- added unit 6 of U1
Connections:
- net FPGA_LED_0 is gone; now on net FMC_NBL1: U1.K19 (IO_L13N_T2_MRCC_15)
- net FPGA_LED_1 is gone; now on net FMC_A20: U1.N22 (IO_L15P_T2_DQS_15)
- net FPGA_LED_3 is gone; now on net FMC_A22: U1.L19 (IO_L14P_T2_SRCC_15)
- net FMC_A16: now also U1.C22 (IO_L20P_T3_16); no longer U1.N19 (IO_L17N_T2_A25_15)
- net FMC_A17: now also U1.B22 (IO_L20N_T3_16); no longer U1.K13 (IO_L19P_T3_A22_15)
- net FMC_A18: now also U1.D21 (IO_L23N_T3_16); no longer U1.J16 (IO_0_15)
- net FMC_A19: now also U1.M22 (IO_L15N_T2_DQS_ADV_B_15); no longer U1.J17 (IO_L21N_T3_DQS_A18_15)
- net FMC_A20: no longer U1.L16 (IO_L23P_T3_FOE_B_15)
- net FMC_A21: now also U1.N20 (IO_L18P_T2_A24_15); no longer U1.K16 (IO_L23N_T3_FWE_B_15)
- net FMC_A22: no longer U1.L18 (IO_L16N_T2_A27_15)
- net FMC_A23: now also U1.M21 (IO_L10P_T1_AD11P_15); no longer U1.L13 (IO_L20N_T3_A19_15)
- net FMC_A24: now also U1.K21 (IO_L9P_T1_DQS_AD3P_15); no longer U1.J20 (IO_L11P_T1_SRCC_15)
- net FMC_A25: now also U1.J22 (IO_L7P_T1_AD2P_15); no longer U1.M18 (IO_L16P_T2_A28_15)
- net FMC_AD0: now also U1.D22 (IO_L22N_T3_16); no longer U1.J22 (IO_L7P_T1_AD2P_15)
- net FMC_AD1: now also U1.J14 (IO_L3P_T0_DQS_AD1P_15); no longer U1.L15 (IO_L22N_T3_A16_15)
- net FMC_AD10: now also U1.B21 (IO_L21P_T3_DQS_16); no longer U1.G16 (IO_L2N_T0_AD8N_15)
- net FMC_AD11: now also U1.A19 (IO_L17N_T2_16); no longer U1.H13 (IO_L1P_T0_AD0P_15)
- net FMC_AD12: now also U1.B18 (IO_L11N_T1_SRCC_16); no longer U1.G15 (IO_L2P_T0_AD8P_15)
- net FMC_AD13: now also U1.B20 (IO_L16P_T2_16); no longer U1.G13 (IO_L1N_T0_AD0N_15)
- net FMC_AD14: now also U1.A21 (IO_L21N_T3_DQS_16); no longer U1.K14 (IO_L19N_T3_A21_VREF_15)
- net FMC_AD15: now also U1.A20 (IO_L16N_T2_16); no longer U1.H19 (IO_L12N_T1_MRCC_15)
- net FMC_AD2: now also U1.H19 (IO_L12N_T1_MRCC_15); no longer U1.K21 (IO_L9P_T1_DQS_AD3P_15)
- net FMC_AD3: now also U1.H20 (IO_L8P_T1_AD10P_15); no longer U1.L21 (IO_L10N_T1_AD11N_15)
- net FMC_AD8: now also U1.A18 (IO_L17P_T2_16); no longer U1.G18 (IO_L4N_T0_AD9N_15)
- net FMC_AD9: now also U1.L20 (IO_L14N_T2_SRCC_15); no longer U1.J14 (IO_L3P_T0_DQS_AD1P_15)
- net FMC_NBL0: now also U1.L21 (IO_L10N_T1_AD11N_15); no longer U1.M13 (IO_L20P_T3_A20_15)
- net FMC_NBL1: no longer U1.N18 (IO_L17P_T2_A26_15)
- net FMC_NE1: now also U1.E22 (IO_L22P_T3_16); no longer U1.G20 (IO_L8N_T1_AD10N_15)
- net FMC_NE2: now also U1.J21 (IO_L11N_T1_SRCC_15); no longer U1.M21 (IO_L10P_T1_AD11P_15)
- net FMC_NE3: now also U1.E21 (IO_L23P_T3_16); no longer U1.H22 (IO_L7N_T1_AD2N_15)
- net FMC_NL_NADV: now also U1.K22 (IO_L9N_T1_DQS_AD3N_15); no longer U1.J21 (IO_L11N_T1_SRCC_15)
- net FMC_NOE: now also U1.J20 (IO_L11P_T1_SRCC_15); no longer U1.K17 (IO_L21P_T3_DQS_15)
- net FMC_NWAIT: now also U1.G20 (IO_L8N_T1_AD10N_15); no longer U1.K22 (IO_L9N_T1_DQS_AD3N_15)
- net FMC_NWE: now also U1.H22 (IO_L7N_T1_AD2N_15); no longer U1.H20 (IO_L8P_T1_AD10P_15)
- net GND: now also R24.2
- net MCU_LED_0: now also U2.M1 (PC2); no longer U2.N13 (PH8)
- net MCU_LED_1: now also U2.M2 (PC3); no longer U2.N11 (PF13)
- net MCU_LED_2: now also U2.P1 (PA0); no longer U2.P11 (PF12)
- net MCU_LED_3: now also U2.P2 (PA1); no longer U2.N7 (PF11)
- net FPGA_CLK_25MHZ: no longer names the net of U1.K18 (IO_L13P_T2_MRCC_15)
- net FPGA_LED_2: no longer names the net of U1.M17 (IO_25_15)
- no-connect marks 86 -> 191
Other:
- moved on the sheet: C64, C65, C66, C68, J4, J5, L1, R24, R26, R27, TP1, TP2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

Commit message: Continued line card bringup board
Parts:
- C40, C44: value 2.2 uF -> 4.7 uF; footprint azonenberg_pcb:EIA_0805_CAP_NOSILK -> azonenberg_pcb:EIA_0603_CAP_NOSILK
Connections:
- net FMC_AD1: now also U1.E16 (IO_L5P_T0_16); no longer U1.J14 (IO_L3P_T0_DQS_AD1P_15)
- net FMC_AD4: now also U1.A16 (IO_L9N_T1_DQS_16); no longer U1.H15 (IO_L5N_T0_AD9N_15)
- net FMC_AD5: now also U1.D16 (IO_L5N_T0_16); no longer U1.H14 (IO_L3N_T0_DQS_AD1N_15)
- net FMC_AD6: now also U1.B17 (IO_L11P_T1_SRCC_16); no longer U1.G17 (IO_L4P_T0_AD9P_15)
- net FMC_AD7: now also U1.B16 (IO_L7N_T1_16); no longer U1.H18 (IO_L6N_T0_VREF_15)
- net SFP_MOD_ABS: now also U2.R7 (PA6); no longer U2.N15 (PH12)
- net SFP_RS1: now also U2.C12 (PC10); no longer U2.D12 (PH15)
- net SFP_RX_LOS: now also U2.P8 (PG0); no longer U2.N14 (PH10)
- net SFP_TX_DISABLE: now also U2.R8 (PB0); no longer U2.M13 (PH11)
- net SFP_TX_FAULT: now also U2.P7 (PB2); no longer U2.C13 (PH13)
Changed lines of the file:
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@@
 	)
 	(no_connect
+		(at 356.87 30.48)
+	)
+	(no_connect
 		(at 182.88 111.76)
 	)
@@
 	)
 	(no_connect
+		(at 356.87 35.56)
+	)
+	(no_connect
 		(at 416.56 120.65)
 	)
@@
 	)
 	(no_connect
-		(at 298.45 43.18)
-	)
-	(no_connect
 		(at 356.87 96.52)
 	)
@@
 	)
 	(no_connect
-		(at 298.45 63.5)
-	)
-	(no_connect
 		(at 416.56 204.47)
 	)
@@
 	)
 	(no_connect
-		(at 87.63 36.83)
-	)
-	(no_connect
 		(at 130.81 91.44)
 	)
@@
 	)
 	(no_connect
-		(at 36.83 46.99)
-	)
-	(no_connect
 		(at 298.45 25.4)
 	)
@@
 	)
 	(no_connect
-		(at 87.63 31.75)
+		(at 356.87 43.18)
 	)
 	(no_connect
@@
 	)
 	(no_connect
+		(at 356.87 33.02)
+	)
+	(no_connect
 		(at 416.56 168.91)
 	)
@@
 	)
 	(no_connect
-		(at 130.81 57.15)
-	)
-	(no_connect
 		(at 356.87 20.32)
 	)
@@
 	)
 	(no_connect
+		(at 130.81 116.84)
+	)
+	(no_connect
 		(at 416.56 110.49)
 	)
@@
 	)
 	(no_connect
-		(at 182.88 86.36)
-	)
-	(no_connect
 		(at 298.45 68.58)
 	)
@@
 	)
 	(no_connect
-		(at 298.45 48.26)
-	)
-	(no_connect
 		(at 416.56 191.77)
 	)
@@
 	)
 	(no_connect
-		(at 298.45 40.64)
-	)
-	(no_connect
 		(at 298.45 137.16)
 	)
@@
 	)
 	(no_connect
+		(at 130.81 119.38)
+	)
+	(no_connect
 		(at 416.56 128.27)
 	)
@@
 	)
 	(no_connect
-		(at 416.56 212.09)
+		(at 298.45 48.26)
 	)
 	(no_connect
-		(at 298.45 53.34)
+		(at 416.56 212.09)
 	)
 	(no_connect
@@
 	)
 	(no_connect
+		(at 130.81 111.76)
+	)
+	(no_connect
 		(at 298.45 142.24)
 	)
@@
 	)
 	(no_connect
-		(at 298.45 71.12)
+		(at 130.81 114.3)
 	)
 	(no_connect
@@
 	)
 	(no_connect
+		(at 130.81 124.46)
+	)
+	(no_connect
+		(at 356.87 48.26)
+	)
+	(no_connect
 		(at 36.83 175.26)
 	)
@@
 	)
 	(label "FMC_AD1"
-		(at 356.87 30.48 180)
+		(at 298.45 40.64 180)
 		(fields_autoplaced yes)
 		(effects
@@
 	)
 	(label "FMC_AD5"
-		(at 356.87 33.02 180)
+		(at 298.45 43.18 180)
 		(fields_autoplaced yes)
 		(effects
@@
 	)
 	(label "FMC_AD7"
-		(at 356.87 48.26 180)
+		(at 298.45 53.34 180)
 		(fields_autoplaced yes)
 		(effects
@@
 	)
 	(label "FMC_AD6"
-		(at 356.87 35.56 180)
+		(at 298.45 71.12 180)
 		(fields_autoplaced yes)
 		(effects
@@
 	)
 	(label "FMC_AD4"
-		(at 356.87 43.18 180)
+		(at 298.45 63.5 180)
 		(fields_autoplaced yes)
 		(effects
@@
 	(hierarchical_label "SFP_TX_FAULT"
 		(shape input)
-		(at 130.81 119.38 180)
+		(at 87.63 36.83 180)
 		(fields_autoplaced yes)
 		(effects
@@
 	(hierarchical_label "SFP_RX_LOS"
 		(shape input)
-		(at 130.81 111.76 180)
+		(at 182.88 86.36 180)
 		(fields_autoplaced yes)
 		(effects
@@
 	(hierarchical_label "SFP_TX_DISABLE"
 		(shape output)
-		(at 130.81 114.3 180)
+		(at 87.63 31.75 180)
 		(fields_autoplaced yes)
 		(effects
@@
 	(hierarchical_label "SFP_RS1"
 		(shape output)
-		(at 130.81 124.46 180)
+		(at 130.81 57.15 180)
 		(fields_autoplaced yes)
 		(effects
@@
 	(hierarchical_label "SFP_MOD_ABS"
 		(shape input)
-		(at 130.81 116.84 180)
+		(at 36.83 46.99 180)
 		(fields_autoplaced yes)
 		(effects
@@
 		(fields_autoplaced yes)
 		(property "Reference" "C44"
-			(at 108.331 214.9915 0)
+			(at 108.331 214.6878 0)
 			(effects
 				(font
@@
 			)
 		)
-		(property "Value" "2.2 uF"
-			(at 108.331 217.7666 0)
+		(property "Value" "4.7 uF"
+			(at 108.331 217.1121 0)
 			(effects
 				(font
@@
 			)
 		)
-		(property "Footprint" "azonenberg_pcb:EIA_0805_CAP_NOSILK"
+		(property "Footprint" "azonenberg_pcb:EIA_0603_CAP_NOSILK"
 			(at 106.3752 219.71 0)
 			(effects
@@
 		(fields_autoplaced yes)
 		(property "Reference" "C40"
-			(at 95.631 214.9915 0)
+			(at 95.631 214.6878 0)
 			(effects
 				(font
@@
 			)
 		)
-		(property "Value" "2.2 uF"
-			(at 95.631 217.7666 0)
+		(property "Value" "4.7 uF"
+			(at 95.631 217.1121 0)
 			(effects
 				(font
@@
 			)
 		)
-		(property "Footprint" "azonenberg_pcb:EIA_0805_CAP_NOSILK"
+		(property "Footprint" "azonenberg_pcb:EIA_0603_CAP_NOSILK"
 			(at 93.6752 219.71 0)
 			(effects

Commit message: Finished initial lcbringup test board, ready for review
Parts:
- J5, TP1: footprint azonenberg_pcb:CONN_HEADER_2.54MM_1x3 -> azonenberg_pcb:CONN_HEADER_2.54MM_1x3_REFLOW
Changed lines of the file:
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@@
 			)
 		)
-		(property "Footprint" "azonenberg_pcb:CONN_HEADER_2.54MM_1x3"
+		(property "Footprint" "azonenberg_pcb:CONN_HEADER_2.54MM_1x3_REFLOW"
 			(at 58.42 186.69 0)
 			(effects
@@
 			)
 		)
-		(property "Footprint" "azonenberg_pcb:CONN_HEADER_2.54MM_1x3"
+		(property "Footprint" "azonenberg_pcb:CONN_HEADER_2.54MM_1x3_REFLOW"
 			(at 58.42 196.85 0)
 			(effects
