File: pcb/lcbringup/sfp.kicad_sch (KiCad schematic)
At the start: 23 parts, among them J3 CONN_SFP_HOST, J7 SFP_CAGE, U1 XC7A35T-2FGG484C, U8 SIT9121AI-2BF-XXS156.250000G

Commit message: Continued lcbringup layout
Connections:
- net GTP_REF_N: now also C70.2; no longer C71.2
- net GTP_REF_P: now also C71.2; no longer C70.2
- net SFP_RX_N: now also J3.12 (RX_N); no longer J3.13 (RX_P)
- net SFP_RX_P: now also J3.13 (RX_P); no longer J3.12 (RX_N)
Other:
- note removed: "Pair swap for routing"
- moved on the sheet: C69, C70, C71, U8
Changed lines of the file:
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@@
 	(title_block
 		(title "Andrew D. Zonenberg")
-		(date "2025-01-10")
+		(date "2025-01-14")
 		(rev "0.1")
 		(company "Antikernel Labs")
@@
 	)
 	(junction
-		(at 38.1 77.47)
+		(at 34.29 168.91)
 		(diameter 0)
 		(color 0 0 0 0)
@@
 	)
 	(junction
-		(at 38.1 85.09)
+		(at 34.29 176.53)
 		(diameter 0)
 		(color 0 0 0 0)
@@
 	(wire
 		(pts
-			(xy 38.1 77.47) (xy 38.1 80.01)
+			(xy 34.29 168.91) (xy 34.29 171.45)
 		)
 		(stroke
@@
 	(wire
 		(pts
-			(xy 90.17 76.2) (xy 106.68 76.2)
-		)
-		(stroke
-			(width 0)
-			(type default)
-		)
-	)
-	(wire
-		(pts
-			(xy 38.1 82.55) (xy 38.1 85.09)
-		)
-		(stroke
-			(width 0)
-			(type default)
-		)
-	)
-	(wire
-		(pts
-			(xy 106.68 76.2) (xy 106.68 80.01)
+			(xy 34.29 173.99) (xy 34.29 176.53)
 		)
 		(stroke
@@
 	(wire
 		(pts
-			(xy 68.58 76.2) (xy 68.58 80.01)
+			(xy 64.77 167.64) (xy 64.77 171.45)
 		)
 		(stroke
@@
 	(wire
 		(pts
-			(xy 24.13 77.47) (xy 38.1 77.47)
+			(xy 20.32 168.91) (xy 34.29 168.91)
 		)
 		(stroke
@@
 	(wire
 		(pts
-			(xy 68.58 86.36) (xy 68.58 82.55)
+			(xy 64.77 177.8) (xy 64.77 173.99)
 		)
 		(stroke
@@
 	(wire
 		(pts
-			(xy 90.17 86.36) (xy 106.68 86.36)
-		)
-		(stroke
-			(width 0)
-			(type default)
-		)
-	)
-	(wire
-		(pts
 			(xy 226.06 114.3) (xy 231.14 114.3)
 		)
@@
 	(wire
 		(pts
-			(xy 82.55 86.36) (xy 68.58 86.36)
+			(xy 78.74 177.8) (xy 64.77 177.8)
 		)
 		(stroke
@@
 	(wire
 		(pts
-			(xy 106.68 86.36) (xy 106.68 82.55)
-		)
-		(stroke
-			(width 0)
-			(type default)
-		)
-	)
-	(wire
-		(pts
-			(xy 82.55 76.2) (xy 68.58 76.2)
+			(xy 78.74 167.64) (xy 64.77 167.64)
 		)
 		(stroke
@@
 	(wire
 		(pts
-			(xy 38.1 85.09) (xy 24.13 85.09)
+			(xy 34.29 176.53) (xy 20.32 176.53)
 		)
 		(stroke
@@
 			(width 0)
 			(type default)
-		)
-	)
-	(text "Pair swap for routing"
-		(exclude_from_sim no)
-		(at 227.33 46.99 0)
-		(effects
-			(font
-				(size 1.27 1.27)
-			)
-			(justify right bottom)
 		)
 	)
@@
 	)
 	(label "SFP_RX_P"
-		(at 241.3 49.53 180)
+		(at 241.3 46.99 180)
 		(fields_autoplaced yes)
 		(effects
@@
 		)
 	)
+	(label "GTP_REF_P"
+		(at 86.36 177.8 0)
+		(fields_autoplaced yes)
+		(effects
+			(font
+				(size 1.27 1.27)
+			)
+			(justify left bottom)
+		)
+	)
 	(label "SFP_TX_P"
 		(at 241.3 54.61 180)
@@
 	)
 	(label "GTP_REF_AC_N"
-		(at 68.58 86.36 0)
+		(at 64.77 177.8 0)
 		(fields_autoplaced yes)
 		(effects
@@
 	)
 	(label "GTP_REF_AC_P"
-		(at 68.58 76.2 0)
+		(at 64.77 167.64 0)
 		(fields_autoplaced yes)
 		(effects
@@
 		)
 	)
+	(label "GTP_REF_N"
+		(at 86.36 167.64 0)
+		(fields_autoplaced yes)
+		(effects
+			(font
+				(size 1.27 1.27)
+			)
+			(justify left bottom)
+		)
+	)
 	(label "SFP_RX_N"
-		(at 241.3 46.99 180)
+		(at 241.3 49.53 180)
 		(fields_autoplaced yes)
 		(effects
@@
 	(hierarchical_label "3V3"
 		(shape input)
-		(at 24.13 77.47 180)
+		(at 20.32 168.91 180)
 		(fields_autoplaced yes)
 		(effects
@@
 	(hierarchical_label "GND"
 		(shape input)
-		(at 24.13 85.09 180)
+		(at 20.32 176.53 180)
 		(fields_autoplaced yes)
 		(effects
@@
 	(symbol
 		(lib_id "device:C")
-		(at 86.36 86.36 90)
+		(at 82.55 177.8 90)
 		(unit 1)
 		(exclude_from_sim no)
@@
 		(fields_autoplaced yes)
 		(property "Reference" "C71"
-			(at 86.36 80.0565 90)
+			(at 82.55 171.4965 90)
 			(effects
 				(font
@@
 		)
 		(property "Value" "0.1 uF"
-			(at 86.36 82.4808 90)
+			(at 82.55 173.9208 90)
 			(effects
 				(font
@@
 		)
 		(property "Footprint" "azonenberg_pcb:EIA_0402_CAP_NOSILK"
-			(at 90.17 85.3948 0)
+			(at 86.36 176.8348 0)
 			(effects
 				(font
@@
 		)
 		(property "Datasheet" ""
-			(at 86.36 86.36 0)
+			(at 82.55 177.8 0)
 			(effects
 				(font
@@
 		)
 		(property "Description" "Unpolarized capacitor"
-			(at 86.36 86.36 0)
+			(at 82.55 177.8 0)
 			(effects
 				(font
@@
 	(symbol
 		(lib_id "device:C")
-		(at 86.36 76.2 90)
+		(at 82.55 167.64 90)
 		(unit 1)
 		(exclude_from_sim no)
@@
 		(fields_autoplaced yes)
 		(property "Reference" "C70"
-			(at 86.36 69.8965 90)
+			(at 82.55 161.3365 90)
 			(effects
 				(font
@@
 		)
 		(property "Value" "0.1 uF"
-			(at 86.36 72.3208 90)
+			(at 82.55 163.7608 90)
 			(effects
 				(font
@@
 		)
 		(property "Footprint" "azonenberg_pcb:EIA_0402_CAP_NOSILK"
-			(at 90.17 75.2348 0)
+			(at 86.36 166.6748 0)
 			(effects
 				(font
@@
 		)
 		(property "Datasheet" ""
-			(at 86.36 76.2 0)
+			(at 82.55 167.64 0)
 			(effects
 				(font
@@
 		)
 		(property "Description" "Unpolarized capacitor"
-			(at 86.36 76.2 0)
+			(at 82.55 167.64 0)
 			(effects
 				(font
@@
 	(symbol
 		(lib_id "osc-azonenberg:OSC_LVDS")
-		(at 45.72 86.36 0)
+		(at 41.91 177.8 0)
 		(unit 1)
 		(exclude_from_sim no)
@@
 		(dnp no)
 		(property "Reference" "U8"
-			(at 53.34 71.5696 0)
+			(at 49.53 163.0096 0)
 			(effects
 				(font
@@
 		)
 		(property "Value" "SIT9121AI-2BF-XXS156.250000G"
-			(at 46.736 74.168 0)
+			(at 42.926 165.608 0)
 			(effects
 				(font
@@
 		)
 		(property "Footprint" "azonenberg_pcb:OSCILLATOR_LVDS_3.2x2.5"
-			(at 45.72 86.36 0)
+			(at 41.91 177.8 0)
 			(effects
 				(font
@@
 		)
 		(property "Datasheet" ""
-			(at 45.72 86.36 0)
+			(at 41.91 177.8 0)
 			(effects
 				(font
@@
 		)
 		(property "Description" ""
-			(at 45.72 86.36 0)
+			(at 41.91 177.8 0)
 			(effects
 				(font
@@
 	(symbol
 		(lib_id "device:C")
-		(at 24.13 81.28 0)
+		(at 20.32 172.72 0)
 		(unit 1)
 		(exclude_from_sim no)
@@
 		(fields_autoplaced yes)
 		(property "Reference" "C69"
-			(at 27.051 80.0678 0)
+			(at 23.241 171.5078 0)
 			(effects
 				(font
@@
 		)
 		(property "Value" "0.47 uF"
-			(at 27.051 82.4921 0)
+			(at 23.241 173.9321 0)
 			(effects
 				(font
@@
 		)
 		(property "Footprint" "azonenberg_pcb:EIA_0402_CAP_NOSILK"
-			(at 25.0952 85.09 0)
+			(at 21.2852 176.53 0)
 			(effects
 				(font
@@
 		)
 		(property "Datasheet" ""
-			(at 24.13 81.28 0)
+			(at 20.32 172.72 0)
 			(effects
 				(font
@@
 		)
 		(property "Description" "Unpolarized capacitor"
-			(at 24.13 81.28 0)
-			(effects
-				(font
+			(at 20.32 172.72 0)
+			(effects
+				(font
