File: pcb/dual-sfp28/dual-sfp28.kicad_sch (KiCad schematic)
At the start: 50 parts, among them J1 CONN_01X10, J2 ARF6-08-S-D-A-K-TR, J3 CONN_SFP_HOST_DUAL, J4 SCREWHOLE, M1 LOGO, M2 LOGO, M3 LOGO, U1 TCA6424A

Commit message: Initial versino of dual-sfp28 is fully routed and ready for review
Connections:
- net LED2_P: now also U1.10 (P11); no longer U1.3 (P02)
- net LED3_P: now also U1.9 (P10); no longer U1.4 (P03)
- net SFP0_RX_LOS: now also U1.17 (P20); no longer U1.14 (P15)
- net SFP0_TX_DISABLE: now also U1.4 (P03); no longer U1.10 (P11)
- net SFP0_TX_FAULT: now also U1.3 (P02); no longer U1.9 (P10)
- net SFP1_MOD_ABS: now also U1.8 (P07); no longer U1.21 (P24)
- net SFP1_RX_LOS: now also U1.6 (P05); no longer U1.22 (P25)
- net SFP1_TX_DISABLE: now also U1.11 (P12); no longer U1.18 (P21)
- net SFP1_TX_FAULT: now also U1.12 (P13); no longer U1.17 (P20)
- net at R11.2: now also U1.5 (P04); no longer U1.20 (P23)
- net at R10.2: now also U1.7 (P06); no longer U1.19 (P22)
- net at R6.2: now also U1.16 (P17); no longer U1.11 (P12)
- net at R7.2: now also U1.14 (P15); no longer U1.12 (P13)
Other:
- company: (none) -> Antikernel Labs
- title: (none) -> Dual SFP28 to ARF6/PicoBlade
- moved on the sheet: R10, R11, R6, R7
Changed lines of the file:
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@@
 	(generator_version "8.0")
 	(paper "A3")
+	(title_block
+		(title "Dual SFP28 to ARF6/PicoBlade")
+		(date "2025-05-31")
+		(rev "0.1")
+		(company "Antikernel Labs")
+		(comment 1 "Andrew D. Zonenberg")
+	)
 	(junction
 		(at 67.31 66.04)
@@
 	)
 	(no_connect
+		(at 39.37 167.64)
+	)
+	(no_connect
 		(at 41.91 91.44)
 	)
@@
 	)
 	(no_connect
-		(at 39.37 124.46)
-	)
-	(no_connect
-		(at 39.37 154.94)
-	)
-	(no_connect
 		(at 67.31 91.44)
 	)
 	(no_connect
-		(at 39.37 177.8)
+		(at 39.37 162.56)
 	)
 	(no_connect
@@
 	)
 	(no_connect
-		(at 39.37 129.54)
+		(at 67.31 99.06)
 	)
 	(no_connect
-		(at 67.31 99.06)
+		(at 41.91 99.06)
 	)
 	(no_connect
-		(at 39.37 132.08)
+		(at 41.91 101.6)
 	)
 	(no_connect
-		(at 41.91 99.06)
+		(at 39.37 170.18)
 	)
 	(no_connect
-		(at 39.37 127)
+		(at 39.37 177.8)
 	)
 	(no_connect
-		(at 41.91 101.6)
+		(at 39.37 165.1)
 	)
 	(no_connect
 		(at 39.37 152.4)
 	)
+	(no_connect
+		(at 39.37 172.72)
+	)
 	(wire
 		(pts
-			(xy 229.87 218.44) (xy 241.3 218.44)
+			(xy 30.48 127) (xy 39.37 127)
 		)
 		(stroke
@@
 	(wire
 		(pts
-			(xy 231.14 46.99) (xy 231.14 49.53)
+			(xy 229.87 218.44) (xy 241.3 218.44)
 		)
 		(stroke
@@
 	(wire
 		(pts
-			(xy 38.1 167.64) (xy 39.37 167.64)
+			(xy 231.14 46.99) (xy 231.14 49.53)
 		)
 		(stroke
@@
 	(wire
 		(pts
+			(xy 38.1 124.46) (xy 39.37 124.46)
+		)
+		(stroke
+			(width 0)
+			(type default)
+		)
+	)
+	(wire
+		(pts
 			(xy 52.07 215.9) (xy 54.61 215.9)
 		)
@@
 	(wire
 		(pts
-			(xy 38.1 144.78) (xy 39.37 144.78)
+			(xy 38.1 149.86) (xy 39.37 149.86)
 		)
 		(stroke
@@
 	(wire
 		(pts
-			(xy 121.92 218.44) (xy 124.46 218.44)
+			(xy 38.1 129.54) (xy 39.37 129.54)
 		)
 		(stroke
@@
 	(wire
 		(pts
-			(xy 44.45 194.31) (xy 59.69 194.31)
+			(xy 121.92 218.44) (xy 124.46 218.44)
 		)
 		(stroke
@@
 	(wire
 		(pts
-			(xy 38.1 142.24) (xy 39.37 142.24)
+			(xy 44.45 194.31) (xy 59.69 194.31)
 		)
 		(stroke
@@
 	(wire
 		(pts
-			(xy 151.13 238.76) (xy 162.56 238.76)
+			(xy 38.1 154.94) (xy 39.37 154.94)
 		)
 		(stroke
@@
 	(wire
 		(pts
-			(xy 30.48 170.18) (xy 39.37 170.18)
+			(xy 151.13 238.76) (xy 162.56 238.76)
 		)
 		(stroke
@@
 	(wire
 		(pts
-			(xy 38.1 165.1) (xy 39.37 165.1)
+			(xy 151.13 218.44) (xy 162.56 218.44)
 		)
 		(stroke
@@
 	(wire
 		(pts
-			(xy 151.13 218.44) (xy 162.56 218.44)
+			(xy 30.48 132.08) (xy 39.37 132.08)
 		)
 		(stroke
@@
 	)
 	(label "SFP0_RX_LOS"
-		(at 39.37 149.86 180)
+		(at 39.37 160.02 180)
 		(fields_autoplaced yes)
 		(effects
@@
 	)
 	(label "SFP1_RX_LOS"
-		(at 39.37 172.72 180)
+		(at 30.48 127 180)
 		(fields_autoplaced yes)
 		(effects
@@
 	)
 	(label "SFP1_MOD_ABS"
-		(at 30.48 170.18 180)
+		(at 30.48 132.08 180)
 		(fields_autoplaced yes)
 		(effects
@@
 	)
 	(label "LED2_P"
-		(at 39.37 119.38 180)
+		(at 39.37 139.7 180)
 		(fields_autoplaced yes)
 		(effects
@@
 	)
 	(label "SFP0_RS0"
-		(at 30.48 142.24 180)
+		(at 30.48 154.94 180)
 		(fields_autoplaced yes)
 		(effects
@@
 	)
 	(label "SFP0_TX_DISABLE"
-		(at 39.37 139.7 180)
+		(at 39.37 121.92 180)
 		(fields_autoplaced yes)
 		(effects
@@
 	)
 	(label "SFP1_RS0"
-		(at 30.48 165.1 180)
+		(at 30.48 129.54 180)
 		(fields_autoplaced yes)
 		(effects
@@
 	)
 	(label "SFP0_RS1"
-		(at 30.48 144.78 180)
+		(at 30.48 149.86 180)
 		(fields_autoplaced yes)
 		(effects
@@
 	)
 	(label "SFP1_TX_FAULT"
-		(at 39.37 160.02 180)
+		(at 39.37 144.78 180)
 		(fields_autoplaced yes)
 		(effects
@@
 	)
 	(label "SFP1_RS1"
-		(at 30.48 167.64 180)
+		(at 30.48 124.46 180)
 		(fields_autoplaced yes)
 		(effects
@@
 	)
 	(label "SFP0_TX_FAULT"
-		(at 39.37 137.16 180)
+		(at 39.37 119.38 180)
 		(fields_autoplaced yes)
 		(effects
@@
 	)
 	(label "SFP1_TX_DISABLE"
-		(at 39.37 162.56 180)
+		(at 39.37 142.24 180)
 		(fields_autoplaced yes)
 		(effects
@@
 	)
 	(label "LED3_P"
-		(at 39.37 121.92 180)
+		(at 39.37 137.16 180)
 		(fields_autoplaced yes)
 		(effects
@@
 	(symbol
 		(lib_id "device:R")
-		(at 34.29 167.64 90)
+		(at 34.29 124.46 90)
 		(unit 1)
 		(exclude_from_sim no)
@@
 		(dnp no)
 		(property "Reference" "R11"
-			(at 38.1 166.37 90)
+			(at 38.1 123.19 90)
 			(effects
 				(font
@@
 		)
 		(property "Value" "1K"
-			(at 34.29 167.64 90)
+			(at 34.29 124.46 90)
 			(effects
 				(font
@@
 		)
 		(property "Footprint" "azonenberg_pcb:EIA_0402_RES_NOSILK"
-			(at 34.29 169.418 90)
+			(at 34.29 126.238 90)
 			(effects
 				(font
@@
 		)
 		(property "Datasheet" ""
-			(at 34.29 167.64 0)
+			(at 34.29 124.46 0)
 			(effects
 				(font
@@
 		)
 		(property "Description" "Resistor"
-			(at 34.29 167.64 0)
+			(at 34.29 124.46 0)
 			(effects
 				(font
@@
 	(symbol
 		(lib_id "device:R")
-		(at 34.29 165.1 90)
+		(at 34.29 129.54 90)
 		(unit 1)
 		(exclude_from_sim no)
@@
 		(dnp no)
 		(property "Reference" "R10"
-			(at 38.1 163.83 90)
+			(at 38.1 128.27 90)
 			(effects
 				(font
@@
 		)
 		(property "Value" "1K"
-			(at 34.29 165.1 90)
+			(at 34.29 129.54 90)
 			(effects
 				(font
@@
 		)
 		(property "Footprint" "azonenberg_pcb:EIA_0402_RES_NOSILK"
-			(at 34.29 166.878 90)
+			(at 34.29 131.318 90)
 			(effects
 				(font
@@
 		)
 		(property "Datasheet" ""
-			(at 34.29 165.1 0)
+			(at 34.29 129.54 0)
 			(effects
 				(font
@@
 		)
 		(property "Description" "Resistor"
-			(at 34.29 165.1 0)
+			(at 34.29 129.54 0)
 			(effects
 				(font
@@
 	(symbol
 		(lib_id "device:R")
-		(at 34.29 144.78 90)
+		(at 34.29 149.86 90)
 		(unit 1)
 		(exclude_from_sim no)
@@
 		(dnp no)
 		(property "Reference" "R7"
-			(at 38.1 143.51 90)
+			(at 38.1 148.59 90)
 			(effects
 				(font
@@
 		)
 		(property "Value" "1K"
-			(at 34.29 144.78 90)
+			(at 34.29 149.86 90)
 			(effects
 				(font
@@
 		)
 		(property "Footprint" "azonenberg_pcb:EIA_0402_RES_NOSILK"
-			(at 34.29 146.558 90)
+			(at 34.29 151.638 90)
 			(effects
 				(font
@@
 		)
 		(property "Datasheet" ""
-			(at 34.29 144.78 0)
+			(at 34.29 149.86 0)
 			(effects
 				(font
@@
 		)
 		(property "Description" "Resistor"
-			(at 34.29 144.78 0)
+			(at 34.29 149.86 0)
 			(effects
 				(font
@@
 	(symbol
 		(lib_id "device:R")
-		(at 34.29 142.24 90)
+		(at 34.29 154.94 90)
 		(unit 1)
 		(exclude_from_sim no)
@@
 		(dnp no)
 		(property "Reference" "R6"
-			(at 38.1 140.97 90)
+			(at 38.1 153.67 90)
 			(effects
 				(font
@@
 		)
 		(property "Value" "1K"
-			(at 34.29 142.24 90)
+			(at 34.29 154.94 90)
 			(effects
 				(font
@@
 		)
 		(property "Footprint" "azonenberg_pcb:EIA_0402_RES_NOSILK"
-			(at 34.29 144.018 90)
+			(at 34.29 156.718 90)
 			(effects
 				(font
@@
 		)
 		(property "Datasheet" ""
-			(at 34.29 142.24 0)
+			(at 34.29 154.94 0)
 			(effects
 				(font
@@
 		)
 		(property "Description" "Resistor"
-			(at 34.29 142.24 0)
+			(at 34.29 154.94 0)
 			(effects
 				(font
