File: pcb/switch-engine/psu.kicad_sch (KiCad schematic)
At the start: 117 parts, among them J1 CONN_PCIE_PWR_8PIN, J2 CONN_IBC_MGMT, J3 CONN_01X03, J4 CORTEX_DEBUG_ETM, J5 FAN_01, J6 FAN_01, Q1 SSM6N58NU, SW1 SWITCH, SW2 SWITCH, U1 STM32L431-QFN48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

Commit message: Continued initial schematic work on switch engine
Other:
- note added: "TODO: little LDO for MDIO level shifters"
Changed lines of the file:
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@@
+		)
+	)
+	(text "TODO: little LDO for MDIO level shifters"
+		(exclude_from_sim no)
+		(at 162.56 270.51 0)
+		(effects
+			(font
+				(size 1.27 1.27)
+			)
+			(justify left)
 		)
 	)
@@
 		)
 	)
+	(hierarchical_label "2V5"
+		(shape output)
+		(at 160.02 265.43 0)
+		(fields_autoplaced yes)
+		(effects
+			(font
+				(size 1.27 1.27)
+			)
+			(justify left)
+		)
+	)

Commit message: First iteration of main board PCB schematic is now passing ERC
Parts:
- removed Q1: SSM6N58NU, azonenberg_pcb:DFN_6_0.65MM_2x2MM_GDS, symbol special-azonenberg:SSM6N58NU_DUAL_NMOS
- removed R9: 100K, azonenberg_pcb:EIA_0402_RES_NOSILK, symbol device:R
- removed TP7: CONN_01X03, azonenberg_pcb:CONN_HEADER_2.54MM_1x3_REFLOW, symbol conn:CONN_01X03
- added C146: DNP, azonenberg_pcb:EIA_0402_CAP_NOSILK, symbol device:C
- added C147, C148: 4.7 uF, azonenberg_pcb:EIA_0603_CAP_NOSILK, symbol device:C
- added R93: 10K, azonenberg_pcb:EIA_0402_RES_NOSILK, symbol device:R
- added TP24: U.FL, azonenberg_pcb:CONN_U.FL_TE_1909763-1, symbol conn:CONN_COAXIAL
- added U28: ADP1740ACPZ-2.5-R7, azonenberg_pcb:QFN_16_0.65MM_4x4MM, symbol power-azonenberg:ADP1741
- F1: value 2A -> 3A
Connections:
- net 12V0_EN: now also R30.1, U1.12 (PA2); no longer R37.1
- net 1V8_PGOOD: now also R34.2; no longer R34.1
- net 2V5: now also C148.1, TP24.1 (In), U28.10 (VOUT), U28.11 (VOUT), U28.12 (VOUT), U28.13 (VOUT), U28.14 (VOUT), U28.9 (ADJ)
- net 3V3: now also C147.1, U28.1 (VIN), U28.15 (VIN), U28.16 (VIN), U28.2 (VIN), U28.3 (VIN); no longer R27.2, R30.1
- net 3V3_PGOOD: now also R23.2; no longer R23.1
- net 3V3_SB: now also R23.1, R33.1, R34.1, R93.2; no longer R23.2, R33.2, R34.2
- net FAN1_PWM: no longer U1.12 (PA2)
- net FAN1_TACH: no longer U1.45 (PB8)
- net FAN2_PWM: no longer U1.28 (PB15)
- net FAN2_TACH: no longer U1.29 (PA8)
- net GND: now also R27.2, R30.2, C146.2, C147.2, C148.2, TP24.2 (Ext), U28.6 (GND), U28.PAD (GND)
- net GTY_VCC_PGOOD: now also R33.2; no longer R33.1
- net GTY_VCCAUX_EN_N renamed GTY_VCCAUX_EN
- net GTY_VCCAUX_EN: now also U7.4 (EN)
- removed net GVEN_3V3: R30.2, U7.4 (EN)
- new net: C146.1, U28.7 (SS)
- new net 2V5_EN: R37.1, U1.29 (PA8), U28.4 (EN)
- new net 2V5_PGOOD: R93.1, U1.45 (PB8), U28.5 (PG)
- no-connect marks 5 -> 6
Other:
- note added: "0.85V supply"
- note added: "0.90V supply"
- note added: "1.2V supply"
- note added: "1.8V for GTY PLLs"
- note added: "1.8V supply"
- note added: "2.5V supply"
- note added: "2V5 is just used for PHY MDIO"
- note added: "3.3V supply"
- note added: "Chassis fans"
- note added: "Power inputs"
- note added: "SUPER_I2C ADDRESS MAP * 0x42: IBC MCU * 0x44: PDU IO expander for rail enables and PGOOD * 0x80: 12V0_LC1 INA230 * 0x82: 12V0_LC2 INA230 * 0x84: 12V0_LOGIC INA230 * 0x90: IBC AT30TS74 * 0x92: PDU AT30TS74 MGMT_I2C ADDRESS MAP * 0x40: Supervisor"
- note added: "Supervisor"
- note added: "Test points"
- note removed: "Level shift GTY_VCCAUX_EN to 3.3V levels since EN of ADP1740 should not exceed VIN"
- note removed: "MGMT_I2C ADDRESS MAP * 0x40: Supervisor"
- note removed: "SUPER_I2C ADDRESS MAP * 0x42: IBC MCU * 0x44: PDU IO expander for rail enables and PGOOD * 0x80: 12V0_LC1 INA230 * 0x82: 12V0_LC2 INA230 * 0x84: 12V0_LOGIC INA230 * 0x90: IBC AT30TS74 * 0x92: PDU AT30TS74"
- note removed: "TODO: little LDO for MDIO level shifters"
- company: (none) -> Antikernel Labs
- title: (none) -> LATENTRED Ethernet Switch - Main Board
- moved on the sheet: C1, C10, C11, C12, C13, C14, C15, C16, C17, C18, C19, C2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

Commit message: Finished schematic review
Parts:
- added TP29, TP7: TESTCLIP, symbol conn:CONN_01X01
Connections:
- net GND: now also TP29.1 (P1), TP7.1 (P1)
- net FPGA_INIT_OE: now reaches U1.28 (PB15)
- no-connect marks 6 -> 5
Other:
- note added: "FPGA status lines are 3.3V here Shifted to 1.8V on other sheet"
- note added: "Ground clips"
Changed lines of the file:
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@@
 	)
 	(no_connect
-		(at 330.2 138.43)
-	)
-	(no_connect
 		(at 331.47 179.07)
 	)
@@
 	(wire
 		(pts
+			(xy 140.97 257.81) (xy 140.97 264.16)
+		)
+		(stroke
+			(width 0)
+			(type default)
+		)
+	)
+	(wire
+		(pts
 			(xy 288.29 21.59) (xy 292.1 21.59)
 		)
@@
 		)
 	)
+	(text "FPGA status lines are 3.3V here\nShifted to 1.8V on other sheet"
+		(exclude_from_sim no)
+		(at 358.14 95.25 0)
+		(effects
+			(font
+				(size 1.27 1.27)
+			)
+			(justify left)
+		)
+	)
 	(text "0.85V supply"
 		(exclude_from_sim no)
@@
 		)
 	)
+	(text "Ground clips"
+		(exclude_from_sim no)
+		(at 135.89 281.94 0)
+		(effects
+			(font
+				(size 2.54 2.54)
+			)
+			(justify left)
+		)
+	)
 	(text "Rtrim = 6 / (Vout - 0.6)\n= 6 / (0.9 - 0.6)\n= 20k"
 		(exclude_from_sim no)
@@
 	)
 	(label "GND"
+		(at 140.97 264.16 180)
+		(fields_autoplaced yes)
+		(effects
+			(font
+				(size 1.27 1.27)
+			)
+			(justify right bottom)
+		)
+	)
+	(label "GND"
 		(at 334.01 91.44 0)
 		(fields_autoplaced yes)
@@
 		)
 	)
+	(hierarchical_label "FPGA_INIT_OE"
+		(shape output)
+		(at 330.2 138.43 180)
+		(fields_autoplaced yes)
+		(effects
+			(font
+				(size 1.27 1.27)
+			)
+			(justify right)
+		)
+	)
 	(symbol
 		(lib_id "passive-azonenberg:INDUCTOR_PWROUT")
@@
 	)
 	(symbol
+		(lib_id "conn:CONN_01X01")
+		(at 146.05 264.16 0)
+		(unit 1)
+		(exclude_from_sim no)
+		(in_bom yes)
+		(on_board yes)
+		(dnp no)
+		(fields_autoplaced yes)
+		(property "Reference" "TP29"
+			(at 147.955 262.9478 0)
+			(effects
+				(font
+					(size 1.27 1.27)
+				)
+				(justify left)
+			)
+		)
+		(property "Value" "TESTCLIP"
+			(at 147.955 265.3721 0)
+			(effects
+				(font
+					(size 1.27 1.27)
+				)
+				(justify left)
+			)
+		)
+		(property "Footprint" ""
+			(at 146.05 264.16 0)
+			(effects
+				(font
+					(size 1.27 1.27)
+				)
+				(hide yes)
+			)
+		)
+		(property "Datasheet" ""
+			(at 146.05 264.16 0)
+			(effects
+				(font
+					(size 1.27 1.27)
+				)
+				(hide yes)
+			)
+		)
+		(property "Description" "Connector, single row, 01x01, pin header"
+			(at 146.05 264.16 0)
+			(effects
+				(font
+					(size 1.27 1.27)
+				)
+				(hide yes)
+			)
+		)
+		(pin "1"
+		)
+		(instances
+			(project "switch-engine"
+				(path "/2594b26d-2fe5-4054-81d2-ca5df3747243/a3f84a70-99b8-4382-a9c4-a0362ca53d67"
+					(reference "TP29")
+					(unit 1)
+				)
+			)
+		)
+	)
+	(symbol
 		(lib_id "power-azonenberg:MYMGK00504ERSR")
 		(at 166.37 247.65 0)
@@
 					(unit 1)
 				)
+			)
+		)
+	)
+	(symbol
+		(lib_id "conn:CONN_01X01")
+		(at 146.05 257.81 0)
+		(unit 1)
+		(exclude_from_sim no)
+		(in_bom yes)
+		(on_board yes)
+		(dnp no)
+		(fields_autoplaced yes)
+		(property "Reference" "TP7"
+			(at 147.955 256.5978 0)
+			(effects
+				(font
+					(size 1.27 1.27)
+				)
+				(justify left)
+			)
+		)
+		(property "Value" "TESTCLIP"
+			(at 147.955 259.0221 0)
+			(effects
+				(font
+					(size 1.27 1.27)
+				)
+				(justify left)
+			)
+		)
+		(property "Footprint" ""
+			(at 146.05 257.81 0)
+			(effects
+				(font
+					(size 1.27 1.27)
+				)
+				(hide yes)
+			)
+		)
+		(property "Datasheet" ""
+			(at 146.05 257.81 0)
+			(effects
+				(font
+					(size 1.27 1.27)
+				)
+				(hide yes)
+			)
+		)
+		(property "Description" "Connector, single row, 01x01, pin header"
+			(at 146.05 257.81 0)
+			(effects
+				(font
+					(size 1.27 1.27)
+				)
+				(hide yes)
+			)
+		)
+		(pin "1"
+		)
+		(instances
+			(project "switch-engine"
+				(path "/2594b26d-2fe5-4054-81d2-ca5df3747243/a3f84a70-99b8-4382-a9c4-a0362ca53d67"
+					(reference "TP7")
+					(unit 1)
+				)

Commit message: Added footprints and created initial skeleton of layout
Parts:
- TP29, TP7: footprint (none) -> azonenberg_pcb:TESTPOINT_SMT_KEYSTONE_5016
Changed lines of the file:
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@@
 			)
 		)
-		(property "Footprint" ""
+		(property "Footprint" "azonenberg_pcb:TESTPOINT_SMT_KEYSTONE_5016"
 			(at 146.05 264.16 0)
 			(effects
@@
 			)
 		)
-		(property "Footprint" ""
+		(property "Footprint" "azonenberg_pcb:TESTPOINT_SMT_KEYSTONE_5016"
 			(at 146.05 257.81 0)
 			(effects
