File: pcb/switch-engine/sfps.kicad_sch (KiCad schematic)
At the start: 13 parts, among them J11 SMPM, J21 ARF6-08-S-D-A-K-TR, J22 ARF6-08-S-D-A-K-TR, J23 CONN_01X10, J24 SMPM, U25 SIT9121AI-2BF-XXS156.250000G, U8 XCKU5P-2FFVB676I

Commit message: Routed line card management low-speed signals
Connections:
- net RC2_N: now also C141.1; no longer C142.1
- net RC2_P: now also C142.1; no longer C141.1
Other:
- moved on the sheet: C141, C142
Changed lines of the file:
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@@
 	(title_block
 		(title "LATENTRED Ethernet Switch - Main Board")
-		(date "2025-06-07")
+		(date "2025-06-11")
 		(rev "0.1")
 		(company "Antikernel Labs")
@@
 	)
 	(label "SFP28_REFCLK_AC_P"
-		(at 91.44 247.65 0)
+		(at 91.44 257.81 0)
 		(fields_autoplaced yes)
 		(effects
@@
 	)
 	(label "SFP28_REFCLK_AC_N"
-		(at 91.44 257.81 0)
+		(at 91.44 247.65 0)
 		(fields_autoplaced yes)
 		(effects
@@
 	(symbol
 		(lib_id "device:C")
-		(at 87.63 247.65 90)
+		(at 87.63 257.81 90)
 		(unit 1)
 		(exclude_from_sim no)
@@
 		(fields_autoplaced yes)
 		(property "Reference" "C141"
-			(at 87.63 241.7912 90)
+			(at 87.63 251.9512 90)
 			(effects
 				(font
@@
 		)
 		(property "Value" "0.1 uF"
-			(at 87.63 244.3281 90)
+			(at 87.63 254.4881 90)
 			(effects
 				(font
@@
 		)
 		(property "Footprint" "azonenberg_pcb:EIA_0402_CAP_NOSILK"
-			(at 91.44 246.6848 0)
+			(at 91.44 256.8448 0)
 			(effects
 				(font
@@
 		)
 		(property "Datasheet" ""
-			(at 87.63 247.65 0)
+			(at 87.63 257.81 0)
 			(effects
 				(font
@@
 		)
 		(property "Description" ""
-			(at 87.63 247.65 0)
+			(at 87.63 257.81 0)
 			(effects
 				(font
@@
 	(symbol
 		(lib_id "device:C")
-		(at 87.63 257.81 90)
+		(at 87.63 247.65 90)
 		(unit 1)
 		(exclude_from_sim no)
@@
 		(fields_autoplaced yes)
 		(property "Reference" "C142"
-			(at 87.63 251.9512 90)
+			(at 87.63 241.7912 90)
 			(effects
 				(font
@@
 		)
 		(property "Value" "0.1 uF"
-			(at 87.63 254.4881 90)
+			(at 87.63 244.3281 90)
 			(effects
 				(font
@@
 		)
 		(property "Footprint" "azonenberg_pcb:EIA_0402_CAP_NOSILK"
-			(at 91.44 256.8448 0)
+			(at 91.44 246.6848 0)
 			(effects
 				(font
@@
 		)
 		(property "Datasheet" ""
-			(at 87.63 257.81 0)
+			(at 87.63 247.65 0)
 			(effects
 				(font
@@
 		)
 		(property "Description" ""
-			(at 87.63 257.81 0)
-			(effects
-				(font
+			(at 87.63 247.65 0)
+			(effects
+				(font

Commit message: Continued SERDES SI tuning
Connections:
- net GTY2_RX_N: now also J22.3 (RX0_P); no longer J22.5 (RX0_N)
- net GTY2_RX_P: now also J22.5 (RX0_N); no longer J22.3 (RX0_P)
- net GTY3_RX_N: now also J22.9 (RX1_P); no longer J22.11 (RX1_N)
- net GTY3_RX_P: now also J22.11 (RX1_N); no longer J22.9 (RX1_P)
